Commit message: changed wheel joint types from revolute to fixed

File: robot_model/mp_400/xacros/mp_400_wheel_left.xacro (robot description, xacro)
@@ -2,5 +2,5 @@
 <robot xmlns:xacro="http://www.ros.org/wiki/xacro" name="mp_400">
   <xacro:macro name="wheel_left" params="name parent *origin">
-   <joint name="${name}_joint" type="revolute">
+   <joint name="${name}_joint" type="fixed">
     <xacro:insert_block name="origin" />
     <axis xyz="1 0 0" />

File: robot_model/mp_400/xacros/mp_400_wheel_right.xacro (robot description, xacro)
@@ -2,5 +2,5 @@
 <robot xmlns:xacro="http://www.ros.org/wiki/xacro" name="mp_400">
   <xacro:macro name="wheel_right" params="name parent *origin">
-   <joint name="${name}_joint" type="revolute">
+   <joint name="${name}_joint" type="fixed">
     <xacro:insert_block name="origin" />
     <axis xyz="1 0 0" />
