Commit message: robot model update + added the cpr_node + unwanted_joint_state_publisher removed

File: robot_model/mp_400/xacros/igus_5DOF_SV.xacro (robot description, xacro)
@@ -9,5 +9,5 @@
       <limit effort="30" velocity="1.0" />
     </joint>
-    <joint name="arm_joint" type="prismatic">
+    <joint name="arm_joint" type="fixed">
       <parent link="linear_link" />
       <child link = "igus_base_link" />

Commit message: Update the link lengths

File: robot_model/mp_400/xacros/igus_5DOF_SV.xacro (robot description, xacro)
@@ -9,8 +9,8 @@
       <limit effort="30" velocity="1.0" />
     </joint>
-    <joint name="arm_joint" type="fixed">
+    <joint name="arm_joint" type="prismatic">
       <parent link="linear_link" />
       <child link = "igus_base_link" />
-      <origin xyz="0.0 -0.148 0.0" rpy="3.14 0 1.57" />
+      <origin xyz="0.0 -0.21 -0.055" rpy="3.14 0 1.57" />
       <axis xyz="-1 0 0"/>
       <limit effort="100" velocity="1.0" lower = "0.0" upper = "1.0"/>
@@ -130,5 +130,5 @@
     <parent link="igus_base_link"/>
     <child link="link1"/>
-    <origin rpy="0 0 0" xyz="0 0 0.1275"/>
+    <origin rpy="0 0 0" xyz="0 0 0.25"/>
     <limit effort="100" velocity="30"/>
     <joint_properties damping="0.0" friction="0.0"/>
@@ -143,13 +143,13 @@
   </joint>
  <joint name="joint3" type="continuous">
-    <axis xyz="0 1 0"/>
+    <axis xyz="0 -1 0"/>
     <parent link="link2"/>
     <child link="link3"/>
-    <origin rpy="0 1.57079632679 0" xyz="0 0 0.270"/>
+    <origin rpy="0 1.57079632679 0" xyz="0 0 0.355"/>
     <limit effort="100" velocity="30"/>
     <joint_properties damping="0.0" friction="0.0"/>
   </joint>
  <joint name="joint4" type="continuous">
-    <axis xyz="0 1 0"/>
+    <axis xyz="0 -1 0"/>
     <parent link="link3"/>
     <child link="link4"/>

Commit message: updated URDF

File: robot_model/mp_400/xacros/igus_5DOF_SV.xacro (robot description, xacro)
@@ -12,7 +12,7 @@
       <parent link="linear_link" />
       <child link = "igus_base_link" />
-      <origin xyz="0.0 -0.21 -0.055" rpy="3.14 0 1.57" />
+      <origin xyz="0.0 -0.36 -0.055" rpy="3.14 0 1.57" />
       <axis xyz="-1 0 0"/>
-      <limit effort="100" velocity="1.0" lower = "0.0" upper = "1.0"/>
+      <limit effort="100" velocity="0.025" lower = "0.0" upper = "0.95"/>
       <dynamics damping="1000.0"/>
     </joint>
@@ -38,5 +38,5 @@
   <link name="igus_base_link">
     <visual>
-	  <origin rpy="0 0 0" xyz="0 0 0"/>
+    <origin rpy="0 0 0" xyz="0 0 0"/>
       <geometry>
           <mesh filename="package://neo_mp_400/robot_model/mp_400/meshes/Joint0.dae"  scale="0.001 0.001 0.001"/>
@@ -58,5 +58,5 @@
   <link name="link1">
     <visual>
-    <origin rpy="0 0 0" xyz="0 0 0"/>
+    <origin rpy="0 0 0" xyz="0.01 0 -0.01"/>
       <geometry>
           <mesh filename="package://neo_mp_400/robot_model/mp_400/meshes/Joint1.dae"  scale="0.001 0.001 0.001"/>
@@ -66,11 +66,17 @@
       <origin xyz="0 0 0" rpy="0 0 0" />
       <geometry>
-          <mesh filename="package://neo_mp_400/robot_model/mp_400/meshes/Joint1Coll.dae" scale="0.001 0.001 0.001"/>
-        </geometry>
-    </collision>
+          <mesh filename="package://neo_mp_400/robot_model/mp_400/meshes/Joint1.dae" scale="0.001 0.001 0.001"/>
+        </geometry>
+    </collision>
+<inertial>
+      <origin xyz="0.0 0.0 0.0" rpy="0 0 0"/>
+      <mass value="5.0"/>
+      <inertia ixx="0.1045" ixy="-0.000460884801" ixz="0.000101130383"
+                    iyy="0.105" iyz="0.002941" izz="0.01284"/>
+    </inertial>
   </link>
   <link name="link2">
     <visual>
-    <origin rpy="0 0 0" xyz="0 0 0"/>
+    <origin rpy="0 0 0" xyz="0.01 0 -0.01"/>
       <geometry>
           <mesh filename="package://neo_mp_400/robot_model/mp_400/meshes/Joint2.dae"  scale="0.001 0.001 0.001"/>
@@ -80,11 +86,17 @@
       <origin xyz="0 0 0" rpy="0 0 0" />
       <geometry>
-          <mesh filename="package://neo_mp_400/robot_model/mp_400/meshes/Joint2Coll.dae" scale="0.001 0.001 0.001"/>
-        </geometry>
-    </collision>
+          <mesh filename="package://neo_mp_400/robot_model/mp_400/meshes/Joint2.dae" scale="0.001 0.001 0.001"/>
+        </geometry>
+    </collision>
+<inertial>
+      <origin xyz="0.0 0.0 0.0" rpy="0 0 0"/>
+      <mass value="5.0"/>
+      <inertia ixx="0.1045" ixy="-0.000460884801" ixz="0.000101130383"
+                    iyy="0.105" iyz="0.002941" izz="0.01284"/>
+    </inertial>
   </link>
   <link name="link3">
     <visual>
-    <origin rpy="0 0 0" xyz="0 0 0"/>
+    <origin rpy="0 0 0" xyz="0.01 0 0"/>
       <geometry>
           <mesh filename="package://neo_mp_400/robot_model/mp_400/meshes/Joint3.dae"  scale="0.001 0.001 0.001"/>
@@ -94,5 +106,5 @@
       <origin xyz="0 0 0" rpy="0 0 0" />
       <geometry>
-          <mesh filename="package://neo_mp_400/robot_model/mp_400/meshes/Joint3Coll.dae" scale="0.001 0.001 0.001"/>
+          <mesh filename="package://neo_mp_400/robot_model/mp_400/meshes/Joint3.dae" scale="0.001 0.001 0.001"/>
         </geometry>
     </collision>
@@ -100,5 +112,5 @@
   <link name="link4">
     <visual>
-    <origin rpy="0 0 0" xyz="0 0 0"/>
+    <origin rpy="0 0 0" xyz="0 0 0.0"/>
       <geometry>
           <mesh filename="package://neo_mp_400/robot_model/mp_400/meshes/Joint4.dae"  scale="0.001 0.001 0.001"/>
@@ -108,5 +120,5 @@
       <origin xyz="0 0 0" rpy="0 0 0" />
       <geometry>
-          <mesh filename="package://neo_mp_400/robot_model/mp_400/meshes/Joint4Coll.dae" scale="0.001 0.001 0.001"/>
+          <mesh filename="package://neo_mp_400/robot_model/mp_400/meshes/Joint4.dae" scale="0.001 0.001 0.001"/>
         </geometry>
     </collision>
@@ -114,5 +126,5 @@
   <link name="link5">
     <visual>
-    <origin rpy="0 0 0" xyz="0 0 -0.0045"/>
+    <origin rpy="0 0 0" xyz="0 0 -0.025"/>
       <geometry>
           <mesh filename="package://neo_mp_400/robot_model/mp_400/meshes/Joint5.dae"  scale="0.001 0.001 0.001"/>
@@ -122,55 +134,77 @@
       <origin xyz="0 0 0" rpy="0 0 -0.0045" />
       <geometry>
-          <mesh filename="package://neo_mp_400/robot_model/mp_400/meshes/Joint5Coll.dae" scale="0.001 0.001 0.001"/>
-        </geometry>
-    </collision>
-  </link>
-  <joint name="joint1" type="continuous">
+          <mesh filename="package://neo_mp_400/robot_model/mp_400/meshes/Joint5.dae" scale="0.001 0.001 0.001"/>
+        </geometry>
+    </collision>
+  </link>
+  <link name="link6">
+    <visual>
+    <origin rpy="0 0 0" xyz="0 0 -0.04"/>
+      <geometry>
+          <mesh filename="package://neo_mp_400/robot_model/mp_400/meshes/Joint6.dae"  scale="0.001 0.001 0.001"/>
+        </geometry>
+    </visual>
+    <collision>
+      <origin xyz="0 0 0" rpy="0 0 -0.04" />
+      <geometry>
+          <mesh filename="package://neo_mp_400/robot_model/mp_400/meshes/Joint6.dae" scale="0.001 0.001 0.001"/>
+        </geometry>
+    </collision>
+  </link>
+  <joint name="joint1" type="revolute">
     <axis xyz="0 0 1"/>
     <parent link="igus_base_link"/>
     <child link="link1"/>
-    <origin rpy="0 0 0" xyz="0 0 0.25"/>
-    <limit effort="100" velocity="30"/>
-    <joint_properties damping="0.0" friction="0.0"/>
-  </joint>
- <joint name="joint2" type="continuous">
+    <origin rpy="0 0 0" xyz="0 0 0.251"/>
+      <limit effort="100" velocity="1.0" lower = "-2.53" upper = "2.53"/>
+    <joint_properties damping="0.0" friction="0.0"/>
+  </joint>
+ <joint name="joint2" type="revolute">
     <axis xyz="0 1 0"/>
     <parent link="link1"/>
     <child link="link2"/>
     <origin rpy="0 0 0" xyz="0 0 0.10025"/>
-    <limit effort="100" velocity="30"/>
-    <joint_properties damping="0.0" friction="0.0"/>
-  </joint>
- <joint name="joint3" type="continuous">
+      <limit effort="100" velocity="1.0" lower = "-0.785398" upper = "1.22173"/>
+    <joint_properties damping="0.0" friction="0.0"/>
+  </joint>
+ <joint name="joint3" type="revolute">
     <axis xyz="0 -1 0"/>
     <parent link="link2"/>
     <child link="link3"/>
     <origin rpy="0 1.57079632679 0" xyz="0 0 0.355"/>
-    <limit effort="100" velocity="30"/>
-    <joint_properties damping="0.0" friction="0.0"/>
-  </joint>
- <joint name="joint4" type="continuous">
+      <limit effort="100" velocity="1.0" lower = "-1.5708" upper = "1.0472"/>
+    <joint_properties damping="0.0" friction="0.0"/>
+  </joint>
+ <joint name="joint4" type="revolute">
     <axis xyz="0 -1 0"/>
     <parent link="link3"/>
     <child link="link4"/>
-    <origin rpy="0 0 0" xyz="0 0 0.240"/>
-    <limit effort="100" velocity="30"/>
-    <joint_properties damping="0.0" friction="0.0"/>
-  </joint>
- <joint name="joint5" type="continuous">
+    <origin rpy="0 0 0" xyz="0 0 0.274"/>
+      <limit effort="100" velocity="1.0" lower = "-0.523599" upper = "2.0944"/>
+    <joint_properties damping="0.0" friction="0.0"/>
+  </joint>
+ <joint name="joint5" type="revolute">
     <axis xyz="0 0 1"/>
     <parent link="link4"/>
     <child link="link5"/>
     <origin rpy="0 0 0" xyz="0 0 0.1835"/>
-    <limit effort="100" velocity="30"/>
-    <joint_properties damping="0.0" friction="0.0"/>
-  </joint>
-  <transmission name="tran_prismatic">
+      <limit effort="100" velocity="1.0" lower = "-2.96706" upper = "2.96706"/>
+    <joint_properties damping="0.0" friction="0.0"/>
+  </joint>
+ <joint name="joint6" type="revolute">
+    <axis xyz="0 0 1"/>
+    <parent link="link5"/>
+    <child link="link6"/>
+    <origin rpy="0 0 0" xyz="0.0 0 0.095"/>
+      <limit effort="100" velocity="1.0" lower = "-2.96706" upper = "2.96706"/>
+    <joint_properties damping="0.0" friction="0.0"/>
+  </joint>
+   <transmission name="tran_prismatic">
     <type>transmission_interface/SimpleTransmission</type>
     <joint name="arm_joint">
-      <hardwareInterface>hardware_interface/PositionJointInterface</hardwareInterface>
+      <hardwareInterface>hardware_interface/VelocityJointInterface</hardwareInterface>
     </joint>
     <actuator name="tran_prismatic_motor">
-      <mechanicalReduction>1</mechanicalReduction>
+      <mechanicalReduction>15</mechanicalReduction>
     </actuator>
   </transmission>
@@ -178,8 +212,8 @@
     <type>transmission_interface/SimpleTransmission</type>
     <joint name="joint1">
-      <hardwareInterface>hardware_interface/PositionJointInterface</hardwareInterface>
+      <hardwareInterface>hardware_interface/VelocityJointInterface</hardwareInterface>
     </joint>
     <actuator name="tran_roll_motor">
-      <mechanicalReduction>1</mechanicalReduction>
+      <mechanicalReduction>50</mechanicalReduction>
     </actuator>
   </transmission>
@@ -187,8 +221,8 @@
     <type>transmission_interface/SimpleTransmission</type>
     <joint name="joint2">
-      <hardwareInterface>hardware_interface/PositionJointInterface</hardwareInterface>
+      <hardwareInterface>hardware_interface/VelocityJointInterface</hardwareInterface>
     </joint>
     <actuator name="tran_1_motor">
-      <mechanicalReduction>1</mechanicalReduction>
+      <mechanicalReduction>50</mechanicalReduction>
     </actuator>
   </transmission>
@@ -196,8 +230,8 @@
     <type>transmission_interface/SimpleTransmission</type>
     <joint name="joint3">
-      <hardwareInterface>hardware_interface/PositionJointInterface</hardwareInterface>
+      <hardwareInterface>hardware_interface/VelocityJointInterface</hardwareInterface>
     </joint>
     <actuator name="tran_2_motor">
-      <mechanicalReduction>1</mechanicalReduction>
+      <mechanicalReduction>-38</mechanicalReduction>
     </actuator>
   </transmission>
@@ -205,8 +239,8 @@
     <type>transmission_interface/SimpleTransmission</type>
     <joint name="joint4">
-      <hardwareInterface>hardware_interface/PositionJointInterface</hardwareInterface>
+      <hardwareInterface>hardware_interface/VelocityJointInterface</hardwareInterface>
     </joint>
     <actuator name="tran_3_motor">
-      <mechanicalReduction>1</mechanicalReduction>
+      <mechanicalReduction>-38</mechanicalReduction>
     </actuator>
   </transmission>
@@ -214,64 +248,19 @@
     <type>transmission_interface/SimpleTransmission</type>
     <joint name="joint5">
-      <hardwareInterface>hardware_interface/PositionJointInterface</hardwareInterface>
+      <hardwareInterface>hardware_interface/VelocityJointInterface</hardwareInterface>
     </joint>
     <actuator name="tran_4_motor">
-      <mechanicalReduction>1</mechanicalReduction>
-    </actuator>
-  </transmission>
-    <gazebo reference="linear_link">
-            <material>Gazebo/Grey</material>
-            <kp>1000000</kp>
-            <kd>1000000</kd>
-            <mu1>500</mu1>
-            <mu2>200</mu2>
-        </gazebo>
-    <gazebo reference="igus_base_link">
-            <material>Gazebo/Grey</material>
-            <kp>1000000</kp>
-            <kd>1000000</kd>
-            <mu1>1</mu1>
-            <mu2>1</mu2>
-        </gazebo>
-        <!-- Link1 -->
-        <gazebo reference="link1">
-            <material>Gazebo/White</material>
-            <kp>1000000</kp>
-            <kd>1000000</kd>
-            <mu1>0.2</mu1>
-            <mu2>0.2</mu2>
-        </gazebo>
-        <!-- Link2 -->
-        <gazebo reference="link2">
-            <material>Gazebo/White</material>
-            <kp>1000000</kp>
-            <kd>1000000</kd>
-            <mu1>0.2</mu1>
-            <mu2>0.2</mu2>
-        </gazebo>
-        <!-- Link3 -->
-        <gazebo reference="link3">
-            <material>Gazebo/White</material>
-           <kp>1000000</kp>
-            <kd>1000000</kd>
-            <mu1>0.2</mu1>
-            <mu2>0.2</mu2>
-        </gazebo>
-        <!-- Link4 -->
-        <gazebo reference="link4">
-            <material>Gazebo/White</material>
-            <kp>1000000</kp>
-            <kd>1000000</kd>
-            <mu1>0.2</mu1>
-            <mu2>0.2</mu2>
-        </gazebo>
-        <!-- Link5 -->
-        <gazebo reference="link5">
-            <material>Gazebo/White</material>
-            <kp>1000000</kp>
-            <kd>1000000</kd>
-            <mu1>0.2</mu1>
-            <mu2>0.2</mu2>
-        </gazebo>
+      <mechanicalReduction>-28</mechanicalReduction>
+    </actuator>
+  </transmission>
+  <transmission name="tran_5">
+    <type>transmission_interface/SimpleTransmission</type>
+    <joint name="joint6">
+      <hardwareInterface>hardware_interface/VelocityJointInterface</hardwareInterface>
+    </joint>
+    <actuator name="tran_5_motor">
+      <mechanicalReduction>32</mechanicalReduction>
+    </actuator>
+  </transmission>
     </xacro:macro>
 </robot>

Commit message: updated the URDF for the kinematics

File: robot_model/mp_400/xacros/igus_5DOF_SV.xacro (robot description, xacro)
@@ -12,5 +12,5 @@
       <parent link="linear_link" />
       <child link = "igus_base_link" />
-      <origin xyz="0.0 -0.36 -0.055" rpy="3.14 0 1.57" />
+      <origin xyz="0.0 -0.36 -0.0" rpy="3.14 0 1.57" />
       <axis xyz="-1 0 0"/>
       <limit effort="100" velocity="0.025" lower = "0.0" upper = "0.95"/>
@@ -46,5 +46,5 @@
       <origin xyz="0 0 0" rpy="0 0 0" />
       <geometry>
-          <mesh filename="package://neo_mp_400/robot_model/mp_400/meshes/Joint0Coll.dae" scale="0.001 0.001 0.001"/>
+          <mesh filename="package://neo_mp_400/robot_model/mp_400/meshes/Joint0.dae" scale="0.001 0.001 0.001"/>
         </geometry>
     </collision>
@@ -58,5 +58,5 @@
   <link name="link1">
     <visual>
-    <origin rpy="0 0 0" xyz="0.01 0 -0.01"/>
+    <origin rpy="0 0 0" xyz="0.0 0 0.0"/>
       <geometry>
           <mesh filename="package://neo_mp_400/robot_model/mp_400/meshes/Joint1.dae"  scale="0.001 0.001 0.001"/>
@@ -78,5 +78,5 @@
   <link name="link2">
     <visual>
-    <origin rpy="0 0 0" xyz="0.01 0 -0.01"/>
+    <origin rpy="0 0 0" xyz="0.0 0 0.0"/>
       <geometry>
           <mesh filename="package://neo_mp_400/robot_model/mp_400/meshes/Joint2.dae"  scale="0.001 0.001 0.001"/>
@@ -98,5 +98,5 @@
   <link name="link3">
     <visual>
-    <origin rpy="0 0 0" xyz="0.01 0 0"/>
+    <origin rpy="0 0 0" xyz="0.0 0 0"/>
       <geometry>
           <mesh filename="package://neo_mp_400/robot_model/mp_400/meshes/Joint3.dae"  scale="0.001 0.001 0.001"/>
@@ -112,5 +112,5 @@
   <link name="link4">
     <visual>
-    <origin rpy="0 0 0" xyz="0 0 0.0"/>
+    <origin rpy="0 0 0" xyz="0.0 0 0.0"/>
       <geometry>
           <mesh filename="package://neo_mp_400/robot_model/mp_400/meshes/Joint4.dae"  scale="0.001 0.001 0.001"/>
@@ -126,5 +126,5 @@
   <link name="link5">
     <visual>
-    <origin rpy="0 0 0" xyz="0 0 -0.025"/>
+    <origin rpy="0 0 0" xyz="0 0 -0.0"/>
       <geometry>
           <mesh filename="package://neo_mp_400/robot_model/mp_400/meshes/Joint5.dae"  scale="0.001 0.001 0.001"/>
@@ -132,5 +132,5 @@
     </visual>
     <collision>
-      <origin xyz="0 0 0" rpy="0 0 -0.0045" />
+      <origin xyz="0 0 0" rpy="0 0 -0.0" />
       <geometry>
           <mesh filename="package://neo_mp_400/robot_model/mp_400/meshes/Joint5.dae" scale="0.001 0.001 0.001"/>
@@ -140,13 +140,13 @@
   <link name="link6">
     <visual>
-    <origin rpy="0 0 0" xyz="0 0 -0.04"/>
-      <geometry>
-          <mesh filename="package://neo_mp_400/robot_model/mp_400/meshes/Joint6.dae"  scale="0.001 0.001 0.001"/>
-        </geometry>
-    </visual>
-    <collision>
-      <origin xyz="0 0 0" rpy="0 0 -0.04" />
-      <geometry>
-          <mesh filename="package://neo_mp_400/robot_model/mp_400/meshes/Joint6.dae" scale="0.001 0.001 0.001"/>
+      <origin rpy="0.0 0 0" xyz="0 0 0"/>
+      <geometry>
+        <cylinder length="0.03" radius="0.035"/>
+      </geometry>
+    </visual>
+    <collision>
+      <origin xyz="0 0 0" rpy="0 0 -0.0" />
+      <geometry>
+        <cylinder length="0.03" radius="0.035"/>
         </geometry>
     </collision>
@@ -156,5 +156,5 @@
     <parent link="igus_base_link"/>
     <child link="link1"/>
-    <origin rpy="0 0 0" xyz="0 0 0.251"/>
+    <origin rpy="0 0 0" xyz="0 0 0.185"/>
       <limit effort="100" velocity="1.0" lower = "-2.53" upper = "2.53"/>
     <joint_properties damping="0.0" friction="0.0"/>
@@ -164,31 +164,32 @@
     <parent link="link1"/>
     <child link="link2"/>
-    <origin rpy="0 0 0" xyz="0 0 0.10025"/>
-      <limit effort="100" velocity="1.0" lower = "-0.785398" upper = "1.22173"/>
-    <joint_properties damping="0.0" friction="0.0"/>
-  </joint>
- <joint name="joint3" type="revolute">
-    <axis xyz="0 -1 0"/>
+    <origin rpy="0 0 0" xyz="0 0 0.145"/>
+    <limit effort="100" lower="-0.785398" upper="1.22173" velocity="5"/>
+    <dynamics damping="15.0" friction="11"/>
+    <dynamics damping="100.0"/>
+  </joint>
+  <joint name="joint3" type="revolute">
+    <axis xyz="0 1 0"/>
     <parent link="link2"/>
     <child link="link3"/>
-    <origin rpy="0 1.57079632679 0" xyz="0 0 0.355"/>
-      <limit effort="100" velocity="1.0" lower = "-1.5708" upper = "1.0472"/>
-    <joint_properties damping="0.0" friction="0.0"/>
-  </joint>
- <joint name="joint4" type="revolute">
-    <axis xyz="0 -1 0"/>
+    <origin rpy="0 1.57079632679 0" xyz="0 0 0.350"/>
+    <limit effort="100" lower="-1.5708" upper="2.00713" velocity="5"/>
+    <dynamics damping="15.0" friction="11"/>
+  </joint>
+  <joint name="joint4" type="revolute">
+    <axis xyz="0 1 0"/>
     <parent link="link3"/>
     <child link="link4"/>
-    <origin rpy="0 0 0" xyz="0 0 0.274"/>
-      <limit effort="100" velocity="1.0" lower = "-0.523599" upper = "2.0944"/>
-    <joint_properties damping="0.0" friction="0.0"/>
-  </joint>
- <joint name="joint5" type="revolute">
+    <origin rpy="0 0 0" xyz="0 0 0.270"/>
+    <limit effort="100" lower="-0.523599" upper="2.0944" velocity="5"/>
+    <dynamics damping="15.0" friction="11"/>
+  </joint>
+  <joint name="joint5" type="revolute">
     <axis xyz="0 0 1"/>
     <parent link="link4"/>
     <child link="link5"/>
-    <origin rpy="0 0 0" xyz="0 0 0.1835"/>
-      <limit effort="100" velocity="1.0" lower = "-2.96706" upper = "2.96706"/>
-    <joint_properties damping="0.0" friction="0.0"/>
+    <origin rpy="0 0 0" xyz="0 0 0.190"/>
+    <limit effort="100" lower="-0.174533" upper="0.174533" velocity="5"/>
+    <dynamics damping="15.0" friction="11"/>
   </joint>
  <joint name="joint6" type="revolute">
@@ -196,9 +197,9 @@
     <parent link="link5"/>
     <child link="link6"/>
-    <origin rpy="0 0 0" xyz="0.0 0 0.095"/>
-      <limit effort="100" velocity="1.0" lower = "-2.96706" upper = "2.96706"/>
+    <origin rpy="0 0 0" xyz="0.0 0 0.06"/>
+      <limit effort="100" velocity="1.0" lower = "-3.14" upper = "3.14"/>
     <joint_properties damping="0.0" friction="0.0"/>
   </joint>
-   <transmission name="tran_prismatic">
+    <transmission name="tran_prismatic">
     <type>transmission_interface/SimpleTransmission</type>
     <joint name="arm_joint">

Commit message: URDF update

File: robot_model/mp_400/xacros/igus_5DOF_SV.xacro (robot description, xacro)
@@ -156,5 +156,5 @@
     <parent link="igus_base_link"/>
     <child link="link1"/>
-    <origin rpy="0 0 0" xyz="0 0 0.185"/>
+    <origin rpy="0 0 0" xyz="-0.05 0 0.185"/>
       <limit effort="100" velocity="1.0" lower = "-2.53" upper = "2.53"/>
     <joint_properties damping="0.0" friction="0.0"/>
@@ -170,5 +170,5 @@
   </joint>
   <joint name="joint3" type="revolute">
-    <axis xyz="0 1 0"/>
+    <axis xyz="0 -1 0"/>
     <parent link="link2"/>
     <child link="link3"/>
@@ -178,5 +178,5 @@
   </joint>
   <joint name="joint4" type="revolute">
-    <axis xyz="0 1 0"/>
+    <axis xyz="0 -1 0"/>
     <parent link="link3"/>
     <child link="link4"/>
@@ -197,5 +197,5 @@
     <parent link="link5"/>
     <child link="link6"/>
-    <origin rpy="0 0 0" xyz="0.0 0 0.06"/>
+    <origin rpy="0 1.57 0" xyz="-0.04 0 0.04"/>
       <limit effort="100" velocity="1.0" lower = "-3.14" upper = "3.14"/>
     <joint_properties damping="0.0" friction="0.0"/>
