Commit message: urdf update + setting velocity limits

File: robot_model/mp_400/xacros/igus_5DOF_SV.xacro (robot description, xacro)
@@ -12,7 +12,7 @@
       <parent link="linear_link" />
       <child link = "igus_base_link" />
-      <origin xyz="0.0 -0.36 -0.0" rpy="3.14 0 1.57" />
+      <origin xyz="0.0 -0.28 -0.0" rpy="3.14 0 1.57" />
       <axis xyz="-1 0 0"/>
-      <limit effort="100" velocity="0.025" lower = "0.0" upper = "0.95"/>
+      <limit effort="100" velocity="0.025" lower = "0.0" upper = "0.75"/>
       <dynamics damping="1000.0"/>
     </joint>
@@ -157,5 +157,5 @@
     <child link="link1"/>
     <origin rpy="0 0 0" xyz="-0.05 0 0.185"/>
-      <limit effort="100" velocity="1.0" lower = "-2.53" upper = "2.53"/>
+      <limit effort="100" velocity="0.785398" lower = "-2.53" upper = "2.53"/>
     <joint_properties damping="0.0" friction="0.0"/>
   </joint>
@@ -165,5 +165,5 @@
     <child link="link2"/>
     <origin rpy="0 0 0" xyz="0 0 0.145"/>
-    <limit effort="100" lower="-0.785398" upper="1.22173" velocity="5"/>
+    <limit effort="100" lower="-0.785398" upper="1.22173" velocity="0.785398"/>
     <dynamics damping="15.0" friction="11"/>
     <dynamics damping="100.0"/>
@@ -174,5 +174,5 @@
     <child link="link3"/>
     <origin rpy="0 1.57079632679 0" xyz="0 0 0.350"/>
-    <limit effort="100" lower="-1.5708" upper="2.00713" velocity="5"/>
+    <limit effort="100" lower="-0.500" upper="1.0" velocity="0.785398"/>
     <dynamics damping="15.0" friction="11"/>
   </joint>
@@ -182,5 +182,5 @@
     <child link="link4"/>
     <origin rpy="0 0 0" xyz="0 0 0.270"/>
-    <limit effort="100" lower="-0.523599" upper="2.0944" velocity="5"/>
+    <limit effort="100" lower="-0.523599" upper="1.5" velocity="1.0472"/>
     <dynamics damping="15.0" friction="11"/>
   </joint>
@@ -190,5 +190,5 @@
     <child link="link5"/>
     <origin rpy="0 0 0" xyz="0 0 0.190"/>
-    <limit effort="100" lower="-0.174533" upper="0.174533" velocity="5"/>
+    <limit effort="100" lower="-0.174533" upper="0.174533" velocity="1.0472"/>
     <dynamics damping="15.0" friction="11"/>
   </joint>
@@ -198,5 +198,5 @@
     <child link="link6"/>
     <origin rpy="0 1.57 0" xyz="-0.04 0 0.04"/>
-      <limit effort="100" velocity="1.0" lower = "-3.14" upper = "3.14"/>
+      <limit effort="100" velocity="0.523599" lower = "-3.14" upper = "3.14"/>
     <joint_properties damping="0.0" friction="0.0"/>
   </joint>

Commit message: update the joint limits

File: robot_model/mp_400/xacros/igus_5DOF_SV.xacro (robot description, xacro)
@@ -157,5 +157,5 @@
     <child link="link1"/>
     <origin rpy="0 0 0" xyz="-0.05 0 0.185"/>
-      <limit effort="100" velocity="0.785398" lower = "-2.53" upper = "2.53"/>
+      <limit effort="100" velocity="0.785398" lower = "-2.44" upper = "2.44"/>
     <joint_properties damping="0.0" friction="0.0"/>
   </joint>
@@ -174,5 +174,5 @@
     <child link="link3"/>
     <origin rpy="0 1.57079632679 0" xyz="0 0 0.350"/>
-    <limit effort="100" lower="-0.500" upper="1.0" velocity="0.785398"/>
+    <limit effort="100" lower="-0.436332" upper="1.57" velocity="0.785398"/>
     <dynamics damping="15.0" friction="11"/>
   </joint>
@@ -182,5 +182,5 @@
     <child link="link4"/>
     <origin rpy="0 0 0" xyz="0 0 0.270"/>
-    <limit effort="100" lower="-0.523599" upper="1.5" velocity="1.0472"/>
+    <limit effort="100" lower="-1.134" upper="1.57" velocity="1.0472"/>
     <dynamics damping="15.0" friction="11"/>
   </joint>
@@ -190,5 +190,5 @@
     <child link="link5"/>
     <origin rpy="0 0 0" xyz="0 0 0.190"/>
-    <limit effort="100" lower="-0.174533" upper="0.174533" velocity="1.0472"/>
+    <limit effort="100" lower="-3.14" upper="3.14" velocity="1.0472"/>
     <dynamics damping="15.0" friction="11"/>
   </joint>
