Commit message: fixed frame name for front scanner and rviz config

File: robot_model/mp_400/mp_400.urdf.xacro (robot description, xacro)
@@ -51,5 +51,5 @@
 	    	<!--box size="0.445 0.277 0.17"/-->
         </geometry>
-        <material name="Neobotix/Yellow" />
+        <material name="Neobotix/Grey" />
       </visual>
       <collision name='body_collision'>

Commit message: added back laserscanner

File: robot_model/mp_400/mp_400.urdf.xacro (robot description, xacro)
@@ -180,3 +180,31 @@
 	  	</collision>
 	</link>
+        <!--+++++++++++++++++++laserscanner_back_joint++++++++++++++++++++++++-->
+        <joint name="laserscanner_back_joint" type="fixed">
+                  <axis xyz="0 1 0" />
+                  <origin xyz="-0.354 0 0.110" rpy="3.14 0 3.14" />
+                  <parent link="base_link"/>
+                  <child link="laserscanner_back_link"/>
+        </joint>
+        <!--+++++++++++++++++++laserscanner_back_link++++++++++++++++++++++++-->
+        <link name="laserscanner_back_link" type="laser">
+                <inertial>
+                        <mass value="0.001" />
+                        <origin xyz="0 0 0" rpy="0 0 0" />
+                        <inertia ixx="0.0001" ixy="0" ixz="0" iyy="0.000001" iyz="0" izz="0.0001" />
+                </inertial>
+                <visual>
+                        <origin xyz="0 0 0" rpy="0 0 -1.57" />
+                        <geometry>
+                                <mesh filename="package://neo_mp_400/robot_model/mp_400/meshes/SICK-S300.STL" />
+                        </geometry>
+                        <material name="Neobotix/Yellow" />
+                </visual>
+                <collision>
+                        <origin xyz="0 0 0" rpy="0 0 0" />
+                        <geometry>
+                        <cylinder length="0.154" radius="0.053" />
+                        </geometry>
+                </collision>
+        </link>
 </robot>

Commit message: added new robot model

File: robot_model/mp_400/mp_400.urdf.xacro (robot description, xacro)
@@ -2,209 +2,38 @@
 <!-- Materials -->
 <robot xmlns:xacro="http://www.ros.org/wiki/xacro" name="mp_400">
-	<material name="Neobotix/Black">
-        <color rgba="0.0 0.0 0.0 1.0"/>
-    </material>
-    <material name="Neobotix/Blue">
-        <color rgba="0.0 0.0 0.8 1.0"/>
-    </material>
-    <material name="Neobotix/Green">
-        <color rgba="0.0 0.8 0.0 1.0"/>
-    </material>
-    <material name="Neobotix/Grey">
-        <color rgba="0.7 0.7 0.7 1.0"/>
-    </material>
-    <material name="Neobotix/Grey2">
-        <color rgba="0.9 0.9 0.9 1.0"/>
-    </material>
-    <material name="Neobotix/Red">
-        <color rgba="0.8 0.0 0.0 1.0"/>
-    </material>
-    <material name="Neobotix/White">
-        <color rgba="1.0 1.0 1.0 1.0"/>
-    </material>
-    <material name="Neobotix/Yellow">
-        <color rgba="1.0 1.0 0 10" />
-    </material>
+<xacro:include filename="$(find neo_simulation)/robots/mp_400/xacros/mp_400_gazebo.xacro" />
 <!--++++++++++++++++++++++++++++++base_link++++++++++++++++++++++++++++++++++++++++++++++++++++-->
 <!--++++++++++++++++++++body++++++++++++++++++++++++++++-->
-	<link name="base_link">
-      <!--inertial>
-        <mass value="67.010" />
-        <origin xyz="0.0 0.0 0.234" rpy="0 0 0"/>
-        <inertia ixx="1417853.715" ixy="17813.155" ixz="-21078.206"
-                 iyy="2030191.708" iyz="-4813.295"
-                 izz="2180211.662" />
-      </inertial-->
-	  <inertial>
-		  <mass value="5.67" />
-		    <origin xyz="0 0 0.0" rpy="0 0 0"/>
-		    <inertia ixx="0.07" ixy="0.0" ixz="0.0"
-		             iyy="0.08" iyz="0.0"
-		             izz="0.1" />
-	  </inertial>
-      <visual name='body'>
-        <!--origin xyz="0.0 0.0 0.234" rpy="0 0 1.57" /--><!-- for cylinder -->
-		<origin xyz="0.0 0.0 0.0" rpy="0 0 1.57" /><!-- for STL -->
-        <geometry>
-            <mesh filename="package://neo_mp_400/robot_model/mp_400/meshes/MP-400-BODY.STL" scale="0.001 0.001 0.001"/>
-	    	<!--cylinder length="0.381" radius="0.2545"/-->
-	    	<!--box size="0.445 0.277 0.17"/-->
-        </geometry>
-        <material name="Neobotix/Grey" />
-      </visual>
-      <collision name='body_collision'>
-        <origin xyz="0.0 0.0 0.234" rpy="0 0 0" />
-        <geometry>
-          <!--box size="0.445 0.277 0.17"/-->
-          <cylinder length="0.381" radius="0.2545"/>
-        </geometry>
-      </collision>
-<!--+++++++++++++++++++castor_front++++++++++++++++++++++++-->
-	<visual name='castor_front_visual'>
-          <origin xyz="0.2 0 0.018" rpy="0 0 0" />
-          <geometry>
-            <sphere radius="0.016"/>
-          </geometry>
-          <material name="Neobotix/Black" />
-      </visual>
-      <collision name='castor_front_collision'>
-	  	<origin xyz="0.2 0 0.018 " rpy="0 0 0" />
-          <geometry>
-            <sphere radius="0.016"/>
-          </geometry>
-    </collision>
-<!--+++++++++++++++++++castor_back++++++++++++++++++++++++-->
-	<visual name='castor_back_visual'>
-          <origin xyz="-0.2 0 0.018" rpy="0 0 0" />
-          <geometry>
-            <sphere radius="0.016"/>
-          </geometry>
-          <material name="Neobotix/Black" />
-      </visual>
-      <collision name='castor_back_collision'>
-	  	<origin xyz="-0.2 0 0.018 " rpy="0 0 0" />
-          <!--pose>0.3 0 -0.12 0 -0 0</pose-->
-          <geometry>
-            <sphere radius="0.016"/>
-          </geometry>
-       </collision>
-    </link>
-<!--+++++++++++++++++++wheel_left_link++++++++++++++++++++++++-->
-<link name="wheel_left_link" type="wheel">
-    <inertial>
-      <mass value="1.5" />
-      <origin xyz="0.0 0.0 -0.016" rpy="0 0 0" />
-      <inertia ixx="0.0051" ixy="0" ixz="0" iyy="0.0051" iyz="0" izz="0.009" />
-    </inertial>
-    <visual>
-     	<origin xyz="0.0 0.0 -0.016" rpy="0 0 0" />
-     	<geometry>
-        	<!--mesh filename="package://neo_robot_descriptions/mp_400/meshes/MP-400-WHEEL.STL" scale="0.001 0.001 0.001"/-->
-			<cylinder radius="0.075" length="0.03"/>
-     	</geometry>
-     	<material name="Neobotix/Black" />
-    </visual>
-    <collision>
-     	<origin xyz="0.0 0.0 -0.016" rpy="0 0 0" />
-     	<geometry>
-        	<cylinder radius="0.075" length="0.03"/>
-     	</geometry>
-    </collision>
-</link>
-<!--+++++++++++++++++++wheel_left_joint++++++++++++++++++++++++-->
-	<joint name="wheel_left_joint" type="revolute">
-		<origin xyz="0 -0.2645 0.075" rpy="0 1.57 1.57" />
-    	<axis xyz="0 0 1"/>
-    	<limit effort="1000.0" lower="-1e+16" upper="1e+16" velocity="3.5"/>
-    	<joint_properties damping="0.0" friction="0.0" />
-    	<parent link="base_link" />
-    	<child link="wheel_left_link" />
-    </joint>
-	<!--+++++++++++++++++++wheel_right_link++++++++++++++++++++++++-->
-	<link name="wheel_right_link" type="wheel">
-		<inertial>
-		  <mass value="1.5" />
-		  <origin xyz="0 0.0 0.016" rpy="0 0 0" />
-		  <inertia ixx="0.0051" ixy="0" ixz="0" iyy="0.0051" iyz="0" izz="0.009" />
-		</inertial>
-		<visual>
-		 	<origin xyz="0 0.0 0.016" rpy="0 0 0" />
-		 	<geometry>
-		    	<!--mesh filename="package://neo_robot_descriptions/mp_400/meshes/MP-400-WHEEL.STL" scale="0.001 0.001 0.001"/-->
-				<cylinder radius="0.075" length="0.03"/>
-		 	</geometry>
-		 	<material name="Neobotix/Black" />
-		</visual>
-		<collision>
-		 	<origin xyz="0.0 0.0 0.016" rpy="0 0 0" />
-		 	<geometry>
-		    	<cylinder radius="0.075" length="0.03"/>
-		 	</geometry>
-		</collision>
-	</link>
-	<!--+++++++++++++++++++wheel_right_joint++++++++++++++++++++++++-->
-	<joint name="wheel_right_joint" type="revolute">
-    	<origin xyz="0 0.2645 0.075" rpy="0 1.57 1.57" />
-    	<axis xyz="0 0 1"/>
-    	<limit effort="1000.0" lower="-1e+16" upper="1e+16" velocity="3.5"/>
-    	<joint_properties damping="0.0" friction="0.0" />
-    	<parent link="base_link" />
-    	<child link="wheel_right_link" />
-    </joint>
-	<!--+++++++++++++++++++laserscanner_front_joint++++++++++++++++++++++++-->
-	<joint name="laserscanner_front_joint" type="fixed">
-		  <axis xyz="0 1 0" />
-		  <origin xyz="0.230 0 0.110" rpy="3.14 0 0" />
-		  <parent link="base_link"/>
-		  <child link="laserscanner_front_link"/>
-	</joint>
-	<!--+++++++++++++++++++laserscanner_front_link++++++++++++++++++++++++-->
-	<link name="laserscanner_front_link" type="laser">
-		<inertial>
-			<mass value="0.001" />
-			<origin xyz="0 0 0" rpy="0 0 0" />
-			<inertia ixx="0.0001" ixy="0" ixz="0" iyy="0.000001" iyz="0" izz="0.0001" />
-	  	</inertial>
-	  	<visual>
-			<origin xyz="0 0 0" rpy="0 0 -1.57" />
-			<geometry>
-		  		<mesh filename="package://neo_mp_400/robot_model/mp_400/meshes/SICK-S300.STL" />
-			</geometry>
-			<material name="Neobotix/Yellow" />
-	  	</visual>
-	  	<collision>
-			<origin xyz="0 0 0" rpy="0 0 0" />
-			<geometry>
-		  	<cylinder length="0.154" radius="0.053" />
-			</geometry>
-	  	</collision>
-	</link>
-        <!--+++++++++++++++++++laserscanner_back_joint++++++++++++++++++++++++-->
-        <joint name="laserscanner_back_joint" type="fixed">
-                  <axis xyz="0 1 0" />
-                  <origin xyz="-0.354 0 0.110" rpy="3.14 0 3.14" />
-                  <parent link="base_link"/>
-                  <child link="laserscanner_back_link"/>
-        </joint>
-        <!--+++++++++++++++++++laserscanner_back_link++++++++++++++++++++++++-->
-        <link name="laserscanner_back_link" type="laser">
-                <inertial>
-                        <mass value="0.001" />
-                        <origin xyz="0 0 0" rpy="0 0 0" />
-                        <inertia ixx="0.0001" ixy="0" ixz="0" iyy="0.000001" iyz="0" izz="0.0001" />
-                </inertial>
-                <visual>
-                        <origin xyz="0 0 0" rpy="0 0 -1.57" />
-                        <geometry>
-                                <mesh filename="package://neo_mp_400/robot_model/mp_400/meshes/SICK-S300.STL" />
-                        </geometry>
-                        <material name="Neobotix/Yellow" />
-                </visual>
-                <collision>
-                        <origin xyz="0 0 0" rpy="0 0 0" />
-                        <geometry>
-                        <cylinder length="0.154" radius="0.053" />
-                        </geometry>
-                </collision>
-        </link>
+<xacro:include filename="$(find neo_simulation)/robots/mp_400/xacros/mp_400_body.xacro" />
+<!--+++++++++++++++++++castor_wheel_link++++++++++++++++++++++++-->
+<xacro:include filename="$(find neo_simulation)/robots/mp_400/xacros/mp_400_caster_wheel.xacro" />
+<!--+++++++++++++++++++left_wheel_link++++++++++++++++++++++++-->
+<xacro:include filename="$(find neo_simulation)/robots/mp_400/xacros/mp_400_fixed_wheel.xacro" />
+  <xacro:mp_400_base name="base_link">
+  </xacro:mp_400_base>
+  <!-- Wheel Macro -->
+  <xacro:caster_wheel name="wheel_front_left" parent="base_link">
+    <origin xyz="0.165 0.155 0.036" rpy="0 0 1.57" />
+  </xacro:caster_wheel>
+  <xacro:caster_wheel name="wheel_back_left" parent="base_link">
+    <origin xyz="-0.220 0.155 0.036" rpy="0 0 1.57" />
+  </xacro:caster_wheel>
+  <xacro:caster_wheel name="wheel_front_right" parent="base_link">
+    <origin xyz="0.165 -0.155 0.036" rpy="0 0 1.57" />
+  </xacro:caster_wheel>
+   <xacro:caster_wheel name="wheel_back_right" parent="base_link">
+    <origin xyz="-0.220 -0.155 0.036" rpy="0 0 1.57" />
+  </xacro:caster_wheel>
+  <xacro:fixed_wheel name="fixed_wheel_right" parent="base_link">
+    <origin xyz="0. -0.26 0.075" rpy="0 0 -1.57" />
+  </xacro:fixed_wheel>
+  <xacro:fixed_wheel name="fixed_wheel_left" parent="base_link">
+    <origin xyz="-0. 0.26 0.075" rpy="0 0 1.57" />
+  </xacro:fixed_wheel>
+  <!--+++++++++++++++++++laserscanner_link++++++++++++++++++++++++-->
+   <!-- SENSORS -->
+  <xacro:include filename="$(find neo_simulation)/robots/mp_400/xacros/sick_laser.xacro" />
+  <xacro:sick_laser_v0 name="laserscanner_1" parent="base_link" ros_topic="sick/scan">
+    <origin xyz="0.230 0 0.110" rpy="0 3.14 3.14" />
+  </xacro:sick_laser_v0>
 </robot>

Commit message: fixed packet names in robot model

File: robot_model/mp_400/mp_400.urdf.xacro (robot description, xacro)
@@ -2,12 +2,12 @@
 <!-- Materials -->
 <robot xmlns:xacro="http://www.ros.org/wiki/xacro" name="mp_400">
-<xacro:include filename="$(find neo_simulation)/robots/mp_400/xacros/mp_400_gazebo.xacro" />
+<xacro:include filename="$(find neo_mp_400)/robot_model/mp_400/xacros/mp_400_gazebo.xacro" />
 <!--++++++++++++++++++++++++++++++base_link++++++++++++++++++++++++++++++++++++++++++++++++++++-->
 <!--++++++++++++++++++++body++++++++++++++++++++++++++++-->
-<xacro:include filename="$(find neo_simulation)/robots/mp_400/xacros/mp_400_body.xacro" />
+<xacro:include filename="$(find neo_mp_400)/robot_model/mp_400/xacros/mp_400_body.xacro" />
 <!--+++++++++++++++++++castor_wheel_link++++++++++++++++++++++++-->
-<xacro:include filename="$(find neo_simulation)/robots/mp_400/xacros/mp_400_caster_wheel.xacro" />
+<xacro:include filename="$(find neo_mp_400)/robot_model/mp_400/xacros/mp_400_caster_wheel.xacro" />
 <!--+++++++++++++++++++left_wheel_link++++++++++++++++++++++++-->
-<xacro:include filename="$(find neo_simulation)/robots/mp_400/xacros/mp_400_fixed_wheel.xacro" />
+<xacro:include filename="$(find neo_mp_400)/robot_model/mp_400/xacros/mp_400_fixed_wheel.xacro" />
   <xacro:mp_400_base name="base_link">
   </xacro:mp_400_base>
@@ -33,5 +33,5 @@
   <!--+++++++++++++++++++laserscanner_link++++++++++++++++++++++++-->
    <!-- SENSORS -->
-  <xacro:include filename="$(find neo_simulation)/robots/mp_400/xacros/sick_laser.xacro" />
+  <xacro:include filename="$(find neo_mp_400)/robot_model/mp_400/xacros/sick_laser.xacro" />
   <xacro:sick_laser_v0 name="laserscanner_1" parent="base_link" ros_topic="sick/scan">
     <origin xyz="0.230 0 0.110" rpy="0 3.14 3.14" />

File: robot_model/mp_400/xacros/mp_400_body.xacro (robot description, xacro)
@@ -13,5 +13,5 @@
       <origin xyz="0.0 0.0 0." rpy="0 0 1.57" />
         <geometry>
-            <mesh filename="package://neo_simulation/robots/mp_400/meshes/MP-400-BODY.dae" scale="0.001 0.001 0.001"/>
+            <mesh filename="package://neo_mp_400/robot_model/mp_400/meshes/MP-400-BODY.dae" scale="0.001 0.001 0.001"/>
         <!--cylinder length="0.381" radius="0.2545"/-->
         <!--box size="0.445 0.277 0.17"/-->
@@ -21,5 +21,5 @@
         <origin xyz="0.0 0.0 0.0" rpy="0 0 1.57" />
         <geometry>
-          <mesh filename="package://neo_simulation/robots/mp_400/meshes/MP-400-BODY.dae" scale="0.001 0.001 0.001"/>
+          <mesh filename="package://neo_mp_400/robot_model/mp_400/meshes/MP-400-BODY.dae" scale="0.001 0.001 0.001"/>
           <!--cylinder length="0.381" radius="0.2545"/-->
         </geometry>

File: robot_model/mp_400/xacros/mp_400_caster_wheel.xacro (robot description, xacro)
@@ -19,5 +19,5 @@
     <origin xyz="0 0 0" rpy="0 0 0" />
     <geometry>
-            <mesh filename="package://neo_simulation/robots/mp_400/meshes/MP-400-CASTER-WHEEL.dae" scale="0.001 0.001 0.001"/>
+            <mesh filename="package://neo_mp_400/robot_model/mp_400/meshes/MP-400-CASTER-WHEEL.dae" scale="0.001 0.001 0.001"/>
     </geometry>
     </visual>
@@ -25,5 +25,5 @@
       <origin xyz="0 0. 0" rpy="0 0 0" />
       <geometry>
-            <mesh filename="package://neo_simulation/robots/mp_400/meshes/MP-400-CASTER-WHEEL.dae" scale="0.001 0.001 0.001"/>
+            <mesh filename="package://neo_mp_400/robot_model/mp_400/meshes/MP-400-CASTER-WHEEL.dae" scale="0.001 0.001 0.001"/>
       </geometry>
     </collision>

File: robot_model/mp_400/xacros/mp_400_fixed_wheel.xacro (robot description, xacro)
@@ -19,5 +19,5 @@
     <origin xyz="0 0 0.0" rpy="0 0 0" />
         <geometry>
-            <mesh filename="package://neo_simulation/robots/mp_400/meshes/MP-400-FIXED-WHEEL.dae" scale="0.001 0.001 0.001"/>
+            <mesh filename="package://neo_mp_400/robot_model/mp_400/meshes/MP-400-FIXED-WHEEL.dae" scale="0.001 0.001 0.001"/>
         </geometry>
       </visual>
@@ -25,5 +25,5 @@
      <origin xyz="0. 0 0" rpy=" 0 0 0" />
       <geometry>
-            <mesh filename="package://neo_simulation/robots/mp_400/meshes/MP-400-FIXED-WHEEL.dae" scale="0.001 0.001 0.001"/>
+            <mesh filename="package://neo_mp_400/robot_model/mp_400/meshes/MP-400-FIXED-WHEEL.dae" scale="0.001 0.001 0.001"/>
       </geometry>
     </collision>

File: robot_model/mp_400/xacros/sick_laser.xacro (robot description, xacro)
@@ -16,7 +16,7 @@
       <visual>
       <!-- SICK S3 sensor: Uncomment/Comment it out if required  -->
-<!--       <origin xyz="0 0 -0.11" rpy="-1.57 0 3.14" />
+       <origin xyz="0 0 -0.11" rpy="-1.57 0 3.14" />
         <geometry>
-        <mesh filename="package://neo_simulation/robots/mp_400/meshes/SICK-S300.dae" scale="0.001 0.001 0.001" />
+        <mesh filename="package://neo_mp_400/robot_model/mp_400/meshes/SICK-S300.dae" scale="0.001 0.001 0.001" />
         </geometry>
       </visual>
@@ -24,11 +24,11 @@
         <origin xyz="0 0 -0.11" rpy="-1.57 0 3.14" />
         <geometry>
-        <mesh filename="package://neo_simulation/robots/mp_400/meshes/SICK-S300.dae" scale="0.001 0.001 0.001" />
+        <mesh filename="package://neo_mp_400/robot_model/mp_400/meshes/SICK-S300.dae" scale="0.001 0.001 0.001" />
         </geometry>
-      </collision> -->
+      </collision>
       <!-- Microscan 3 sensor: Uncomment/Comment it out if required  -->
- <origin xyz="-0.0 0 -0.06" rpy="1.57 0 0" />
+ <!--<origin xyz="-0.0 0 -0.06" rpy="1.57 0 0" />
       <geometry>
-      <mesh filename="package://neo_simulation/robots/mp_400/meshes/SICK-MICROSCAN3.dae" scale="0.001 0.001 0.001" />
+      <mesh filename="package://neo_mp_400/robot_model/mp_400/meshes/SICK-MICROSCAN3.dae" scale="0.001 0.001 0.001" />
       </geometry>
       </visual>
@@ -36,7 +36,7 @@
  <origin xyz="-0.0 0 -0.06" rpy="1.57 0 0" />
       <geometry>
-        <mesh filename="package://neo_simulation/robots/mp_400/meshes/SICK-MICROSCAN3.dae" scale="0.001 0.001 0.001" />
+        <mesh filename="package://neo_mp_400/robot_model/mp_400/meshes/SICK-MICROSCAN3.dae" scale="0.001 0.001 0.001" />
         </geometry>
-      </collision>
+      </collision> -->
     </link>
   </xacro:macro>

Commit message: added new LiDAR structure, added IMU and ultra sonic links to robot model, added launch file for robot model

File: robot_model/mp_400/mp_400.urdf.xacro (robot description, xacro)
@@ -31,9 +31,81 @@
     <origin xyz="-0. 0.26 0.075" rpy="0 0 1.57" />
   </xacro:fixed_wheel>
-  <!--+++++++++++++++++++laserscanner_link++++++++++++++++++++++++-->
-   <!-- SENSORS -->
+  <!--+++++++++++++++++++ LiDAR ++++++++++++++++++++++++-->
+  <!-- SENSORS -->
   <xacro:include filename="$(find neo_mp_400)/robot_model/mp_400/xacros/sick_laser.xacro" />
-  <xacro:sick_laser_v0 name="laser_1" parent="base_link" ros_topic="laser_1/scan">
+  <xacro:sick_laser_v0 name="lidar_1" parent="base_link" ros_topic="laser_1/scan">
     <origin xyz="0.230 0 0.110" rpy="0 3.14 3.14" />
   </xacro:sick_laser_v0>
+  <!--+++++++++++++++++++ IMU ++++++++++++++++++++++++-->
+  <!-- SENSORS -->
+  <xacro:include filename="$(find neo_mp_400)/robot_model/mp_400/xacros/imu.xacro" />
+  <xacro:imu name="imu_1" parent="base_link">
+    <origin xyz="0.100 0 0.300" rpy="0 0 3.14" />
+  </xacro:imu>
+  <!--+++++++++++++++++++ Ultra Sonic ++++++++++++++++++++++++-->
+  <xacro:include filename="$(find neo_mp_400)/robot_model/mp_400/xacros/ultrasonic.xacro" />
+  <!-- SENSOR 1 -->
+  <!-- xacro:us_sensor name="us_1" parent="base_link">
+    <origin xyz="0.100 0 0.300" rpy="0 3.14 3.14" />
+  </xacro:us_sensor-->
+  <!-- SENSOR 2 -->
+  <!-- xacro:us_sensor name="us_2" parent="base_link">
+    <origin xyz="0.110 0 0.300" rpy="0 3.14 3.14" />
+  </xacro:us_sensor-->
+  <!-- SENSOR 3 -->
+  <!-- xacro:us_sensor name="us_3" parent="base_link">
+    <origin xyz="0.120 0 0.300" rpy="0 3.14 3.14" />
+  </xacro:us_sensor-->
+  <!-- SENSOR 4 -->
+  <!-- xacro:us_sensor name="us_4" parent="base_link">
+    <origin xyz="0.130 0 0.300" rpy="0 3.14 3.14" />
+  </xacro:us_sensor-->
+  <!-- SENSOR 5 -->
+  <!-- xacro:us_sensor name="us_5" parent="base_link">
+    <origin xyz="0.140 0 0.300" rpy="0 3.14 3.14" />
+  </xacro:us_sensor-->
+  <!-- SENSOR 6 -->
+  <!-- xacro:us_sensor name="us_6" parent="base_link">
+    <origin xyz="0.150 0 0.300" rpy="0 3.14 3.14" />
+  </xacro:us_sensor-->
+  <!-- SENSOR 7 -->
+  <!-- xacro:us_sensor name="us_7" parent="base_link">
+    <origin xyz="0.160 0 0.300" rpy="0 3.14 3.14" />
+  </xacro:us_sensor-->
+  <!-- SENSOR 8 -->
+  <!-- xacro:us_sensor name="us_8" parent="base_link">
+    <origin xyz="0.170 0 0.300" rpy="0 3.14 3.14" />
+  </xacro:us_sensor-->
+  <!-- SENSOR 9 -->
+  <!-- xacro:us_sensor name="us_9" parent="base_link">
+    <origin xyz="0.180 0 0.300" rpy="0 3.14 3.14" />
+  </xacro:us_sensor-->
+  <!-- SENSOR 10 -->
+  <!-- xacro:us_sensor name="us_10" parent="base_link">
+    <origin xyz="0.100 0 0.300" rpy="0 3.14 3.14" />
+  </xacro:us_sensor-->
+  <!-- SENSOR 11 -->
+  <!-- xacro:us_sensor name="us_11" parent="base_link">
+    <origin xyz="0.100 0 0.300" rpy="0 3.14 3.14" />
+  </xacro:us_sensor-->
+  <!-- SENSOR 12 -->
+  <!-- xacro:us_sensor name="us_12" parent="base_link">
+    <origin xyz="0.190 0 0.300" rpy="0 3.14 3.14" />
+  </xacro:us_sensor-->
+  <!-- SENSOR 13 -->
+  <!-- xacro:us_sensor name="us_13" parent="base_link">
+    <origin xyz="0.200 0 0.300" rpy="0 3.14 3.14" />
+  </xacro:us_sensor-->
+  <!-- SENSOR 14 -->
+  <!-- xacro:us_sensor name="us_14" parent="base_link">
+    <origin xyz="0.210 0 0.300" rpy="0 3.14 3.14" />
+  </xacro:us_sensor-->
+  <!-- SENSOR 15 -->
+  <!-- xacro:us_sensor name="us_15" parent="base_link">
+    <origin xyz="0.220 0 0.300" rpy="0 3.14 3.14" />
+  </xacro:us_sensor-->
+  <!-- SENSOR 16 -->
+  <!-- xacro:us_sensor name="us_16" parent="base_link">
+    <origin xyz="0.230 0 0.300" rpy="0 3.14 3.14" />
+  </xacro:us_sensor-->
 </robot>
