Commit message: Robot model updated

File: robot_model/mp_400/mp_400.urdf.xacro (robot description, xacro)
@@ -1,4 +1,3 @@
 <?xml version="1.0"?>
-<!-- Materials -->
 <robot xmlns:xacro="http://www.ros.org/wiki/xacro" name="mp_400">
 <xacro:include filename="$(find neo_mp_400)/robot_model/mp_400/xacros/mp_400_gazebo.xacro" />
@@ -9,5 +8,16 @@
 <xacro:include filename="$(find neo_mp_400)/robot_model/mp_400/xacros/mp_400_caster_wheel.xacro" />
 <!--+++++++++++++++++++left_wheel_link++++++++++++++++++++++++-->
-<xacro:include filename="$(find neo_mp_400)/robot_model/mp_400/xacros/mp_400_fixed_wheel.xacro" />
+<xacro:include filename="$(find neo_mp_400)/robot_model/mp_400/xacros/mp_400_fixed_wheel_left.xacro" />
+<!--+++++++++++++++++++right_wheel_link++++++++++++++++++++++++-->
+<xacro:include filename="$(find neo_mp_400)/robot_model/mp_400/xacros/mp_400_fixed_wheel_right.xacro" />
+<!-- SENSORS -->
+<!-- Sick S300 - Comment/Uncomment if required  -->
+<!-- <xacro:include filename="$(find neo_mp_400)/robot_model/mp_400/xacros/sick_S300.xacro" /> -->
+<!-- Microscan - Comment/Uncomment if required -->
+ <xacro:include filename="$(find neo_mp_400)/robot_model/mp_400/urdf//micro_scan.xacro" />
+<!-- USS and IMU - Comment/Uncomment if required  -->
+<!-- <xacro:include filename="$(find neo_mp_400)/robot_model/mp_400/xacros/imu.xacro" />
+<xacro:include filename="$(find neo_mp_400)/robot_model/mp_400/xacros/ultrasonic.xacro" /> -->
+<!-- Base link macro -->
   <xacro:mp_400_base name="base_link">
   </xacro:mp_400_base>
@@ -25,24 +35,21 @@
     <origin xyz="-0.220 -0.155 0.036" rpy="0 0 1.57" />
   </xacro:caster_wheel>
-  <xacro:fixed_wheel name="fixed_wheel_right" parent="base_link">
-    <origin xyz="0. -0.26 0.075" rpy="0 0 -1.57" />
-  </xacro:fixed_wheel>
-  <xacro:fixed_wheel name="fixed_wheel_left" parent="base_link">
-    <origin xyz="-0. 0.26 0.075" rpy="0 0 1.57" />
-  </xacro:fixed_wheel>
-  <!--+++++++++++++++++++ LiDAR ++++++++++++++++++++++++-->
-  <!-- SENSORS -->
-  <xacro:include filename="$(find neo_mp_400)/robot_model/mp_400/xacros/sick_laser.xacro" />
-  <xacro:sick_laser_v0 name="lidar_1" parent="base_link" ros_topic="laser_1/scan">
+  <xacro:fixed_wheel_right name="fixed_wheel_right" parent="base_link">
+    <origin xyz="0. -0.26 0.074" rpy="0 0 1.57" />
+  </xacro:fixed_wheel_right>
+  <xacro:fixed_wheel_left name="fixed_wheel_left" parent="base_link">
+    <origin xyz="-0. 0.26 0.074" rpy="0 0 1.57" />
+  </xacro:fixed_wheel_left>
+  <!--+++++++++++++++++++laserscanner_link++++++++++++++++++++++++-->
+  <xacro:sick_laser_v0 name="lidar_1" parent="base_link" ros_topic="lidar_1/scan_filtered">
     <origin xyz="0.230 0 0.110" rpy="0 3.14 3.14" />
   </xacro:sick_laser_v0>
-  <!--+++++++++++++++++++ IMU ++++++++++++++++++++++++-->
-  <!-- SENSORS -->
-  <xacro:include filename="$(find neo_mp_400)/robot_model/mp_400/xacros/imu.xacro" />
-  <xacro:imu name="imu_1" parent="base_link">
+     <!--+++++++++++++++++++ IMU ++++++++++++++++++++++++-->
+ <!-- Comment or uncomment based on your requirement -->
+<!--   <xacro:imu name="imu_1" parent="base_link">
     <origin xyz="0.100 0 0.300" rpy="0 0 3.14" />
-  </xacro:imu>
+  </xacro:imu> -->
   <!--+++++++++++++++++++ Ultra Sonic ++++++++++++++++++++++++-->
-  <xacro:include filename="$(find neo_mp_400)/robot_model/mp_400/xacros/ultrasonic.xacro" />
+  <!-- Comment or uncomment based on your requirement -->
   <!-- SENSOR 1 -->
   <!-- xacro:us_sensor name="us_1" parent="base_link">
@@ -109,3 +116,7 @@
     <origin xyz="0.230 0 0.300" rpy="0 3.14 3.14" />
   </xacro:us_sensor-->
+    <!--Camera  -->
+<!-- <xacro:camera name="camera" parent="base_link">
+    <origin xyz="0 0 0.38" rpy="0 0 0" />
+  </xacro:camera> -->
 </robot>

File: robot_model/mp_400/xacros/mp_400_body.xacro (robot description, xacro)
@@ -3,5 +3,5 @@
   <xacro:macro name="mp_400_base" params="name">
     <link name="${name}">
-    <inertial>
+  <inertial>
         <mass value="30" />
         <origin xyz="0 0 0" rpy="0 0 0"/>
@@ -9,11 +9,9 @@
                  iyy="0.8856" iyz="0.0"
                  izz="2.5725" />
-    </inertial>
+</inertial>
       <visual name='body'>
       <origin xyz="0.0 0.0 0." rpy="0 0 1.57" />
         <geometry>
             <mesh filename="package://neo_mp_400/robot_model/mp_400/meshes/MP-400-BODY.dae" scale="0.001 0.001 0.001"/>
-        <!--cylinder length="0.381" radius="0.2545"/-->
-        <!--box size="0.445 0.277 0.17"/-->
         </geometry>
       </visual>
@@ -22,8 +20,16 @@
         <geometry>
           <mesh filename="package://neo_mp_400/robot_model/mp_400/meshes/MP-400-BODY.dae" scale="0.001 0.001 0.001"/>
-          <!--cylinder length="0.381" radius="0.2545"/-->
         </geometry>
       </collision>
     </link>
+  <gazebo reference="${name}">
+    <kp>10000.0</kp>
+    <kd>10.0</kd>
+    <mu1>1.5</mu1>
+    <mu2>1.5</mu2>
+    <fdir1>.1 0 0</fdir1>
+    <maxVel>10.0</maxVel>
+    <minDepth>0.0005</minDepth>
+</gazebo>
   </xacro:macro>
 </robot>

File: robot_model/mp_400/xacros/mp_400_caster_wheel.xacro (robot description, xacro)
@@ -4,6 +4,6 @@
    <joint name="${name}_joint" type="fixed">
     <insert_block name="origin" />
-    <axis xyz="0 1 0" />
-    <joint_properties damping="1" friction="1" />
+    <axis xyz="-1 0 0" />
+    <joint_properties damping="1." friction="1.0" />
     <limit effort="1000.0" lower="-1e+16" upper="1e+16" velocity="3.5"/>
     <parent link="${parent}" />
@@ -11,9 +11,10 @@
    </joint>
    <link name="${name}_link" type="wheel">
-    <inertial>
-      <mass value="3.5" />
-      <origin xyz="0.000000010 -0.045437214 -0.073569633" rpy="0 0 0" />
-      <inertia ixx="13.177588678963057" ixy="-0.00000019386313414965295" ixz="-0.0000007636494859403484" iyy="8.48847991205267" iyz="-2.366298925984707" izz="7.157972023102095" />
-    </inertial>
+   <inertial>
+        <mass value="1.4"/>
+        <inertia ixx="0.00499743171" ixy="0.00000004464" ixz="-0.00000002245"
+                 iyy="0.00499741733" iyz="-0.00000000164"
+                 izz="0.00839239692"/>
+</inertial>
       <visual name='caster_wheel'>
     <origin xyz="0 0 0" rpy="0 0 0" />
@@ -29,4 +30,14 @@
     </collision>
     </link>
+<gazebo reference="${name}_link">
+      <kp>10000.0</kp>
+      <kd>10.0</kd>
+      <mu1>0.5</mu1>
+      <mu2>0.2</mu2>
+      <fdir1>.5 0 0</fdir1>
+      <maxVel>3.0</maxVel>
+      <minDepth>0.00</minDepth>
+      <implicitSpringDamper>3</implicitSpringDamper>
+</gazebo>
   </xacro:macro>
 </robot>

File: robot_model/mp_400/xacros/mp_400_gazebo.xacro (robot description, xacro)
@@ -13,6 +13,6 @@
     <self_collide>false</self_collide>
   </gazebo>
-  <gazebo reference="laserscanner_1_link">
-      <sensor type="ray" name="laserscanner_1_link">
+  <gazebo reference="lidar_1_link">
+      <sensor type="ray" name="lidar_1_link">
           <pose>0 0 0 0 0 0</pose>
           <visualize>false</visualize>
@@ -42,18 +42,132 @@
             </noise>
           </ray>
-          <plugin name="laserscanner_1_link" filename="libgazebo_ros_laser.so">
-            <topicName>sick/scan</topicName>
-            <frameName>laserscanner_1_link</frameName>
+          <plugin name="lidar_1_link" filename="libgazebo_ros_laser.so">
+            <topicName>lidar_1/scan_filtered</topicName>
+            <frameName>lidar_1_link</frameName>
           </plugin>
         </sensor>
   </gazebo>
+    <gazebo reference="imu_1_link">
+    <gravity>true</gravity>
+    <sensor name="imu_sensor" type="imu">
+      <always_on>true</always_on>
+      <update_rate>100</update_rate>
+      <visualize>true</visualize>
+      <topic>__default_topic__</topic>
+      <plugin filename="libgazebo_ros_imu_sensor.so" name="imu_plugin">
+        <topicName>imu</topicName>
+        <bodyName>imu_link</bodyName>
+        <updateRateHZ>10.0</updateRateHZ>
+        <gaussianNoise>0.0</gaussianNoise>
+        <xyzOffset>0 0 0</xyzOffset>
+        <rpyOffset>0 0 0</rpyOffset>
+        <frameName>imu_link</frameName>
+      </plugin>
+      <pose>0 0 0 0 0 0</pose>
+    </sensor>
+  </gazebo>
+  <gazebo reference="us_1_link">
+  <!-- Visuals / Collisions omitted for this example -->
+  <sensor type="ray" name="range">
+    <ray>
+         <scan>
+            <horizontal>
+               <samples>1</samples>
+               <resolution>1.0</resolution>
+               <min_angle>-0.01</min_angle>
+               <max_angle>0.01</max_angle>
+            </horizontal>
+            <vertical>
+               <samples>1</samples>
+               <resolution>1</resolution>
+               <min_angle>-0.01</min_angle>
+               <max_angle>0.01</max_angle>
+            </vertical>
+         </scan>
+         <range>
+            <min>0.01</min>
+            <max>3.75</max>
+            <resolution>0.02</resolution>
+         </range>
+      </ray>
+    <plugin name="libgazebo_ros_range" filename="libgazebo_ros_range.so">
+         <gaussianNoise>0.005</gaussianNoise>
+         <alwaysOn>true</alwaysOn>
+         <updateRate>50</updateRate>
+         <topicName>us_sensor</topicName>
+         <frameName>us_1_link</frameName>
+         <radiation>SONAR</radiation>
+         <fov>0.2967</fov>
+    </plugin>
+  </sensor>
+  </gazebo>
+    <!-- camera -->
+  <gazebo reference="camera_link">
+    <sensor type="camera" name="camera1">
+      <update_rate>30.0</update_rate>
+      <camera name="head">
+        <horizontal_fov>1.3962634</horizontal_fov>
+        <image>
+          <width>800</width>
+          <height>800</height>
+          <format>R8G8B8</format>
+        </image>
+        <clip>
+          <near>0.02</near>
+          <far>300</far>
+        </clip>
+        <noise>
+          <type>gaussian</type>
+          <!-- Noise is sampled independently per pixel on each frame.
+               That pixel's noise value is added to each of its color
+               channels, which at that point lie in the range [0,1]. -->
+          <mean>0.0</mean>
+          <stddev>0.007</stddev>
+        </noise>
+      </camera>
+      <plugin name="camera_controller" filename="libgazebo_ros_camera.so">
+        <alwaysOn>true</alwaysOn>
+        <updateRate>0.0</updateRate>
+        <cameraName>camera1</cameraName>
+        <imageTopicName>image_raw</imageTopicName>
+        <cameraInfoTopicName>camera_info</cameraInfoTopicName>
+        <frameName>camera_link</frameName>
+        <hackBaseline>0.07</hackBaseline>
+        <distortionK1>0.0</distortionK1>
+        <distortionK2>0.0</distortionK2>
+        <distortionK3>0.0</distortionK3>
+        <distortionT1>0.0</distortionT1>
+        <distortionT2>0.0</distortionT2>
+      </plugin>
+    </sensor>
+  </gazebo>
   <gazebo>
-    <plugin name="mp_400_controller" filename="libgazebo_ros_planar_move.so">
-      <commandTopic>cmd_vel</commandTopic>
-      <odometryTopic>odom</odometryTopic>
-      <odometryFrame>odom</odometryFrame>
-      <odometryRate>20.0</odometryRate>
-      <robotBaseFrame>base_link</robotBaseFrame>
+    <plugin name="diff_dirve_controller" filename="libgazebo_ros_diff_drive.so">
+        <alwaysOn>true</alwaysOn>
+        <updateRate>40</updateRate>
+        <legacyMode>false</legacyMode>
+        <torque>5</torque>
+        <leftJoint>fixed_wheel_left_joint</leftJoint>
+        <rightJoint>fixed_wheel_right_joint</rightJoint>
+        <wheelSeparation>0.529</wheelSeparation>
+        <wheelDiameter>0.15</wheelDiameter>
+        <commandTopic>cmd_vel</commandTopic>
+        <rosDebugLevel>na</rosDebugLevel>
+        <odometryTopic>odom</odometryTopic>
+        <odometryFrame>odom</odometryFrame>
+        <robotBaseFrame>base_link</robotBaseFrame>
+        <publishWheelTF>true</publishWheelTF>
+        <publishWheelJointState>true</publishWheelJointState>
+        <wheelAcceleration>6.0</wheelAcceleration>
+        <wheelTorque>5</wheelTorque>
+        <odometrySource>world</odometrySource>
+        <publishTf>1</publishTf>
+        <publishOdomTF>true</publishOdomTF>
     </plugin>
   </gazebo>
+<!-- <gazebo>
+  <plugin name="gazebo_ros_control" filename="libgazebo_ros_control.so">
+    <robotNamespace>/mp_400</robotNamespace>
+  </plugin>
+</gazebo> -->
 </robot>

Commit message: Depreceated tags are removed

File: robot_model/mp_400/mp_400.urdf.xacro (robot description, xacro)
@@ -19,24 +19,26 @@
 <!-- <xacro:include filename="$(find neo_mp_400)/robot_model/mp_400/xacros/imu.xacro" />
 <xacro:include filename="$(find neo_mp_400)/robot_model/mp_400/xacros/ultrasonic.xacro" /> -->
+  <link name="base_link" />
 <!-- Base link macro -->
-  <xacro:mp_400_base name="base_link">
+ <xacro:mp_400_base name="base_footprint" parent="base_link">
+    <origin xyz="0 0 0" rpy="0 0 0" />
   </xacro:mp_400_base>
   <!-- Wheel Macro -->
-  <xacro:caster_wheel name="wheel_front_left" parent="base_link">
+  <xacro:caster_wheel name="wheel_front_left" parent="base_footprint">
     <origin xyz="0.165 0.155 0.036" rpy="0 0 1.57" />
   </xacro:caster_wheel>
-  <xacro:caster_wheel name="wheel_back_left" parent="base_link">
+  <xacro:caster_wheel name="wheel_back_left" parent="base_footprint">
     <origin xyz="-0.220 0.155 0.036" rpy="0 0 1.57" />
   </xacro:caster_wheel>
-  <xacro:caster_wheel name="wheel_front_right" parent="base_link">
+  <xacro:caster_wheel name="wheel_front_right" parent="base_footprint">
     <origin xyz="0.165 -0.155 0.036" rpy="0 0 1.57" />
   </xacro:caster_wheel>
-   <xacro:caster_wheel name="wheel_back_right" parent="base_link">
+   <xacro:caster_wheel name="wheel_back_right" parent="base_footprint">
     <origin xyz="-0.220 -0.155 0.036" rpy="0 0 1.57" />
   </xacro:caster_wheel>
-  <xacro:fixed_wheel_right name="fixed_wheel_right" parent="base_link">
+  <xacro:fixed_wheel_right name="fixed_wheel_right" parent="base_footprint">
     <origin xyz="0. -0.26 0.074" rpy="0 0 1.57" />
   </xacro:fixed_wheel_right>
-  <xacro:fixed_wheel_left name="fixed_wheel_left" parent="base_link">
+  <xacro:fixed_wheel_left name="fixed_wheel_left" parent="base_footprint">
     <origin xyz="-0. 0.26 0.074" rpy="0 0 1.57" />
   </xacro:fixed_wheel_left>

File: robot_model/mp_400/xacros/camera.xacro (robot description, xacro)
@@ -5,5 +5,5 @@
     <joint name="${name}_joint" type="fixed">
       <axis xyz="0 1 0" />
-      <insert_block name="origin" />
+      <xacro:insert_block name="origin" />
       <parent link="${parent}"/>
       <child link="${name}_link"/>

File: robot_model/mp_400/xacros/micro_scan.xacro (robot description, xacro)
@@ -4,5 +4,5 @@
     <joint name="${name}_joint" type="fixed">
       <axis xyz="0 1 0" />
-      <insert_block name="origin" />
+      <xacro:insert_block name="origin" />
       <parent link="${parent}"/>
       <child link="${name}_link"/>

File: robot_model/mp_400/xacros/mp_400_body.xacro (robot description, xacro)
@@ -1,7 +1,15 @@
 <?xml version="1.0"?>
 <robot xmlns:xacro="http://www.ros.org/wiki/xacro" name="mp_400">
-  <xacro:macro name="mp_400_base" params="name">
+  <xacro:macro name="mp_400_base" params="name parent *origin">
+    <joint name="${name}_joint" type="fixed">
+      <xacro:insert_block name="origin" />
+      <axis xyz="0 0 -1" />
+      <!-- <limit effort="1000.0" lower="-1e+16" upper="1e+16" velocity="3.5"/> -->
+      <joint_properties damping="1" friction="1" />
+      <parent link="${parent}" />
+      <child link="${name}" />
+   </joint>
     <link name="${name}">
-  <inertial>
+    <inertial>
         <mass value="30" />
         <origin xyz="0 0 0" rpy="0 0 0"/>
@@ -9,5 +17,5 @@
                  iyy="0.8856" iyz="0.0"
                  izz="2.5725" />
-</inertial>
+    </inertial>
       <visual name='body'>
       <origin xyz="0.0 0.0 0." rpy="0 0 1.57" />

File: robot_model/mp_400/xacros/mp_400_caster_wheel.xacro (robot description, xacro)
@@ -3,5 +3,5 @@
   <xacro:macro name="caster_wheel" params="name parent *origin">
    <joint name="${name}_joint" type="fixed">
-    <insert_block name="origin" />
+    <xacro:insert_block name="origin" />
     <axis xyz="-1 0 0" />
     <joint_properties damping="1." friction="1.0" />

File: robot_model/mp_400/xacros/mp_400_fixed_wheel_left.xacro (robot description, xacro)
@@ -3,5 +3,5 @@
   <xacro:macro name="fixed_wheel_left" params="name parent *origin">
    <joint name="${name}_joint" type="revolute">
-    <insert_block name="origin" />
+    <xacro:insert_block name="origin" />
     <axis xyz="1 0 0" />
     <limit effort="1000.0" lower="-1e+16" upper="1e+16" velocity="3.5"/>

File: robot_model/mp_400/xacros/mp_400_fixed_wheel_right.xacro (robot description, xacro)
@@ -3,5 +3,5 @@
   <xacro:macro name="fixed_wheel_right" params="name parent *origin">
    <joint name="${name}_joint" type="revolute">
-    <insert_block name="origin" />
+    <xacro:insert_block name="origin" />
     <axis xyz="1 0 0" />
     <limit effort="1000.0" lower="-1e+16" upper="1e+16" velocity="3.5"/>

File: robot_model/mp_400/xacros/sick_S300.xacro (robot description, xacro)
@@ -4,5 +4,5 @@
     <joint name="${name}_joint" type="fixed">
       <axis xyz="0 1 0" />
-      <insert_block name="origin" />
+      <xacro:insert_block name="origin" />
       <parent link="${parent}"/>
       <child link="${name}_link"/>

File: robot_model/mp_400/xacros/ultrasonic.xacro (robot description, xacro)
@@ -4,5 +4,5 @@
     <joint name="${name}_joint" type="fixed">
       <axis xyz="0 1 0" />
-      <insert_block name="origin" />
+      <xacro:insert_block name="origin" />
       <parent link="${parent}"/>
       <child link="${name}_link"/>

Commit message: Wheel naming changed - removed the term 'Fixed'

File: robot_model/mp_400/mp_400.urdf.xacro (robot description, xacro)
@@ -8,7 +8,7 @@
 <xacro:include filename="$(find neo_mp_400)/robot_model/mp_400/xacros/mp_400_caster_wheel.xacro" />
 <!--+++++++++++++++++++left_wheel_link++++++++++++++++++++++++-->
-<xacro:include filename="$(find neo_mp_400)/robot_model/mp_400/xacros/mp_400_fixed_wheel_left.xacro" />
+<xacro:include filename="$(find neo_mp_400)/robot_model/mp_400/xacros/mp_400_wheel_left.xacro" />
 <!--+++++++++++++++++++right_wheel_link++++++++++++++++++++++++-->
-<xacro:include filename="$(find neo_mp_400)/robot_model/mp_400/xacros/mp_400_fixed_wheel_right.xacro" />
+<xacro:include filename="$(find neo_mp_400)/robot_model/mp_400/xacros/mp_400_wheel_right.xacro" />
 <!-- SENSORS -->
 <!-- Sick S300 - Comment/Uncomment if required  -->
@@ -25,22 +25,22 @@
   </xacro:mp_400_base>
   <!-- Wheel Macro -->
-  <xacro:caster_wheel name="wheel_front_left" parent="base_footprint">
+  <xacro:caster_wheel name="mp_400_wheel_front_left" parent="base_footprint">
     <origin xyz="0.165 0.155 0.036" rpy="0 0 1.57" />
   </xacro:caster_wheel>
-  <xacro:caster_wheel name="wheel_back_left" parent="base_footprint">
+  <xacro:caster_wheel name="mp_400_wheel_back_left" parent="base_footprint">
     <origin xyz="-0.220 0.155 0.036" rpy="0 0 1.57" />
   </xacro:caster_wheel>
-  <xacro:caster_wheel name="wheel_front_right" parent="base_footprint">
+  <xacro:caster_wheel name="mp_400_wheel_front_right" parent="base_footprint">
     <origin xyz="0.165 -0.155 0.036" rpy="0 0 1.57" />
   </xacro:caster_wheel>
-   <xacro:caster_wheel name="wheel_back_right" parent="base_footprint">
+   <xacro:caster_wheel name="mp_400_wheel_back_right" parent="base_footprint">
     <origin xyz="-0.220 -0.155 0.036" rpy="0 0 1.57" />
   </xacro:caster_wheel>
-  <xacro:fixed_wheel_right name="fixed_wheel_right" parent="base_footprint">
+  <xacro:wheel_right name="mp_400_wheel_right" parent="base_footprint">
     <origin xyz="0. -0.26 0.074" rpy="0 0 1.57" />
-  </xacro:fixed_wheel_right>
-  <xacro:fixed_wheel_left name="fixed_wheel_left" parent="base_footprint">
+  </xacro:wheel_right>
+  <xacro:wheel_left name="mp_400_wheel_left" parent="base_footprint">
     <origin xyz="-0. 0.26 0.074" rpy="0 0 1.57" />
-  </xacro:fixed_wheel_left>
+  </xacro:wheel_left>
   <!--+++++++++++++++++++laserscanner_link++++++++++++++++++++++++-->
   <xacro:sick_laser_v0 name="lidar_1" parent="base_link" ros_topic="lidar_1/scan_filtered">

File: robot_model/mp_400/xacros/mp_400_wheel_left.xacro (robot description, xacro)
@@ -1,5 +1,5 @@
 <?xml version="1.0"?>
 <robot xmlns:xacro="http://www.ros.org/wiki/xacro" name="mp_400">
-  <xacro:macro name="fixed_wheel_right" params="name parent *origin">
+  <xacro:macro name="wheel_left" params="name parent *origin">
    <joint name="${name}_joint" type="revolute">
     <xacro:insert_block name="origin" />
@@ -17,8 +17,8 @@
                  izz="0.00739239692"/>
 </inertial>
-      <visual name='fixed_wheel_right'>
-    <origin xyz="0 0 0.0" rpy="0 0 3.14" />
+      <visual name='fixed_wheel_left'>
+    <origin xyz="0 0 0.0" rpy="0 0 0" />
         <geometry>
-            <mesh filename="package://neo_mp_400/robot_model/mp_400/meshes/MP-400-FIXED-WHEEL-RIGHT.dae" scale="0.001 0.001 0.001"/>
+            <mesh filename="package://neo_mp_400/robot_model/mp_400/meshes/MP-400-FIXED-WHEEL-LEFT.dae" scale="0.001 0.001 0.001"/>
         </geometry>
       </visual>
@@ -31,5 +31,5 @@
 </link>
 <gazebo reference="${name}_link">
-      <kp>600.0</kp> <!-- Partial Ziegler-Nichols method -->
+      <kp>600.0</kp>
       <kd>1465.0</kd>
       <mu1>200</mu1>

File: robot_model/mp_400/xacros/mp_400_wheel_right.xacro (robot description, xacro)
@@ -1,5 +1,5 @@
 <?xml version="1.0"?>
 <robot xmlns:xacro="http://www.ros.org/wiki/xacro" name="mp_400">
-  <xacro:macro name="fixed_wheel_left" params="name parent *origin">
+  <xacro:macro name="wheel_right" params="name parent *origin">
    <joint name="${name}_joint" type="revolute">
     <xacro:insert_block name="origin" />
@@ -17,8 +17,8 @@
                  izz="0.00739239692"/>
 </inertial>
-      <visual name='fixed_wheel_left'>
-    <origin xyz="0 0 0.0" rpy="0 0 0" />
+      <visual name='fixed_wheel_right'>
+    <origin xyz="0 0 0.0" rpy="0 0 3.14" />
         <geometry>
-            <mesh filename="package://neo_mp_400/robot_model/mp_400/meshes/MP-400-FIXED-WHEEL-LEFT.dae" scale="0.001 0.001 0.001"/>
+            <mesh filename="package://neo_mp_400/robot_model/mp_400/meshes/MP-400-FIXED-WHEEL-RIGHT.dae" scale="0.001 0.001 0.001"/>
         </geometry>
       </visual>
@@ -31,5 +31,5 @@
 </link>
 <gazebo reference="${name}_link">
-      <kp>600.0</kp>
+      <kp>600.0</kp> <!-- Partial Ziegler-Nichols method -->
       <kd>1465.0</kd>
       <mu1>200</mu1>
