Commit message: Added nanoscan model in the URDF

File: robot_model/mp_400/mp_400.urdf.xacro (robot description, xacro)
@@ -16,4 +16,6 @@
 <!-- Microscan - Comment/Uncomment if required -->
  <xacro:include filename="$(find neo_mp_400)/robot_model/mp_400/xacros/micro_scan.xacro" />
+<!-- Nanoscan - Comment/Uncomment if required -->
+ <xacro:include filename="$(find neo_mp_400)/robot_model/mp_400/xacros/nano_scan.xacro" />
 <!-- USS and IMU - Comment/Uncomment if required  -->
 <!-- <xacro:include filename="$(find neo_mp_400)/robot_model/mp_400/xacros/imu.xacro" />
@@ -44,6 +46,11 @@
   </xacro:wheel_left>
   <!--+++++++++++++++++++laserscanner_link++++++++++++++++++++++++-->
+<!-- S300 and Microscan -->
+<!--   <xacro:sick_laser_v0 name="lidar_1" parent="base_link" ros_topic="lidar_1/scan_filtered">
+    <origin xyz="0.230 0 0.110" rpy="0 3.14 3.14" />
+  </xacro:sick_laser_v0> -->
+<!-- NanoScan -->
   <xacro:sick_laser_v0 name="lidar_1" parent="base_link" ros_topic="lidar_1/scan_filtered">
-    <origin xyz="0.230 0 0.110" rpy="0 3.14 3.14" />
+    <origin xyz="0.230 0 0.05" rpy="0 3.14 3.14" />
   </xacro:sick_laser_v0>
      <!--+++++++++++++++++++ IMU ++++++++++++++++++++++++-->

Commit message: NanoScan added

File: robot_model/mp_400/mp_400.urdf.xacro (robot description, xacro)
@@ -13,7 +13,9 @@
 <!-- SENSORS -->
 <!-- Sick S300 - Comment/Uncomment if required  -->
-<!-- <xacro:include filename="$(find neo_mp_400)/robot_model/mp_400/xacros/sick_S300.xacro" /> -->
+<xacro:include filename="$(find neo_mp_400)/robot_model/mp_400/xacros/sick_S300.xacro" />
 <!-- Microscan - Comment/Uncomment if required -->
- <xacro:include filename="$(find neo_mp_400)/robot_model/mp_400/xacros/micro_scan.xacro" />
+ <!-- <xacro:include filename="$(find neo_mp_400)/robot_model/mp_400/xacros/micro_scan.xacro" /> -->
+<!-- Nanoscan - Comment/Uncomment if required -->
+ <!-- <xacro:include filename="$(find neo_mp_400)/robot_model/mp_400/xacros/nano_scan.xacro" /> -->
 <!-- USS and IMU - Comment/Uncomment if required  -->
 <!-- <xacro:include filename="$(find neo_mp_400)/robot_model/mp_400/xacros/imu.xacro" />
@@ -44,4 +46,5 @@
   </xacro:wheel_left>
   <!--+++++++++++++++++++laserscanner_link++++++++++++++++++++++++-->
+<!-- S300, NanoScan and Microscan -->
   <xacro:sick_laser_v0 name="lidar_1" parent="base_link" ros_topic="lidar_1/scan_filtered">
     <origin xyz="0.230 0 0.110" rpy="0 3.14 3.14" />

File: robot_model/mp_400/xacros/sick_S300.xacro (robot description, xacro)
@@ -17,5 +17,5 @@
         <origin xyz="0 0 -0.11" rpy="-1.57 0 3.14" />
         <geometry>
-        <mesh filename="package://neo_mp_400/robot_model/mp_400/meshes/SICK-MICROSCAN3.dae" scale="0.001 0.001 0.001" />
+        <mesh filename="package://neo_mp_400/robot_model/mp_400/meshes/SICK-S300.dae" scale="0.001 0.001 0.001" />
         </geometry>
       </visual>
@@ -23,5 +23,5 @@
         <origin xyz="0 0 -0.11" rpy="-1.57 0 3.14" />
         <geometry>
-        <mesh filename="package://neo_mp_400/robot_model/mp_400/meshes/SICK-MICROSCAN3.dae" scale="0.001 0.001 0.001" />
+        <mesh filename="package://neo_mp_400/robot_model/mp_400/meshes/SICK-S300.dae" scale="0.001 0.001 0.001" />
         </geometry>
       </collision>

Commit message: updated mesh

File: robot_model/mp_400/mp_400.urdf.xacro (robot description, xacro)
@@ -21,5 +21,7 @@
 <!-- <xacro:include filename="$(find neo_mp_400)/robot_model/mp_400/xacros/imu.xacro" />
 <xacro:include filename="$(find neo_mp_400)/robot_model/mp_400/xacros/ultrasonic.xacro" /> -->
-  <link name="base_link" />
+<!-- Igus -->
+<xacro:include filename="$(find neo_mp_400)/robot_model/mp_400/xacros/igus_5DOF_SV.xacro" />
+<link name="base_link" />
 <!-- Base link macro -->
  <xacro:mp_400_base name="base_footprint" parent="base_link">
@@ -28,14 +30,14 @@
   <!-- Wheel Macro -->
   <xacro:caster_wheel name="mp_400_wheel_front_left" parent="base_footprint">
-    <origin xyz="0.165 0.155 0.036" rpy="0 0 1.57" />
+    <origin xyz="0.164 0.158 0.036" rpy="0 0 1.57" />
   </xacro:caster_wheel>
   <xacro:caster_wheel name="mp_400_wheel_back_left" parent="base_footprint">
-    <origin xyz="-0.220 0.155 0.036" rpy="0 0 1.57" />
+    <origin xyz="-0.319 0.158 0.036" rpy="0 0 1.57" />
   </xacro:caster_wheel>
   <xacro:caster_wheel name="mp_400_wheel_front_right" parent="base_footprint">
-    <origin xyz="0.165 -0.155 0.036" rpy="0 0 1.57" />
+    <origin xyz="0.164 -0.158 0.036" rpy="0 0 1.57" />
   </xacro:caster_wheel>
    <xacro:caster_wheel name="mp_400_wheel_back_right" parent="base_footprint">
-    <origin xyz="-0.220 -0.155 0.036" rpy="0 0 1.57" />
+    <origin xyz="-0.319 -0.158 0.036" rpy="0 0 1.57" />
   </xacro:caster_wheel>
   <xacro:wheel_right name="mp_400_wheel_right" parent="base_footprint">
@@ -50,4 +52,8 @@
     <origin xyz="0.230 0 0.110" rpy="0 3.14 3.14" />
   </xacro:sick_laser_v0>
+<!-- Igus -->
+<xacro:igus_5DOF_SV parent="base_link" prefix="igus">
+    <origin xyz="0 0 0." rpy="0 0 3.14" />
+  </xacro:igus_5DOF_SV>
      <!--+++++++++++++++++++ IMU ++++++++++++++++++++++++-->
  <!-- Comment or uncomment based on your requirement -->

Commit message: robot model update

File: robot_model/mp_400/mp_400.urdf.xacro (robot description, xacro)
@@ -1,133 +1,267 @@
 <?xml version="1.0"?>
-<robot xmlns:xacro="http://www.ros.org/wiki/xacro" name="mp_400">
-<xacro:include filename="$(find neo_mp_400)/robot_model/mp_400/xacros/mp_400_gazebo.xacro" />
-<!--++++++++++++++++++++++++++++++base_link++++++++++++++++++++++++++++++++++++++++++++++++++++-->
-<!--++++++++++++++++++++body++++++++++++++++++++++++++++-->
-<xacro:include filename="$(find neo_mp_400)/robot_model/mp_400/xacros/mp_400_body.xacro" />
-<!--+++++++++++++++++++castor_wheel_link++++++++++++++++++++++++-->
-<xacro:include filename="$(find neo_mp_400)/robot_model/mp_400/xacros/mp_400_caster_wheel.xacro" />
-<!--+++++++++++++++++++left_wheel_link++++++++++++++++++++++++-->
-<xacro:include filename="$(find neo_mp_400)/robot_model/mp_400/xacros/mp_400_wheel_left.xacro" />
-<!--+++++++++++++++++++right_wheel_link++++++++++++++++++++++++-->
-<xacro:include filename="$(find neo_mp_400)/robot_model/mp_400/xacros/mp_400_wheel_right.xacro" />
-<!-- SENSORS -->
-<!-- Sick S300 - Comment/Uncomment if required  -->
-<xacro:include filename="$(find neo_mp_400)/robot_model/mp_400/xacros/sick_S300.xacro" />
-<!-- Microscan - Comment/Uncomment if required -->
- <!-- <xacro:include filename="$(find neo_mp_400)/robot_model/mp_400/xacros/micro_scan.xacro" /> -->
-<!-- Nanoscan - Comment/Uncomment if required -->
- <!-- <xacro:include filename="$(find neo_mp_400)/robot_model/mp_400/xacros/nano_scan.xacro" /> -->
-<!-- USS and IMU - Comment/Uncomment if required  -->
-<!-- <xacro:include filename="$(find neo_mp_400)/robot_model/mp_400/xacros/imu.xacro" />
-<xacro:include filename="$(find neo_mp_400)/robot_model/mp_400/xacros/ultrasonic.xacro" /> -->
-<!-- Igus -->
-<xacro:include filename="$(find neo_mp_400)/robot_model/mp_400/xacros/igus_5DOF_SV.xacro" />
-<link name="base_link" />
-<!-- Base link macro -->
- <xacro:mp_400_base name="base_footprint" parent="base_link">
-    <origin xyz="0 0 0" rpy="0 0 0" />
-  </xacro:mp_400_base>
-  <!-- Wheel Macro -->
-  <xacro:caster_wheel name="mp_400_wheel_front_left" parent="base_footprint">
-    <origin xyz="0.164 0.158 0.036" rpy="0 0 1.57" />
-  </xacro:caster_wheel>
-  <xacro:caster_wheel name="mp_400_wheel_back_left" parent="base_footprint">
-    <origin xyz="-0.319 0.158 0.036" rpy="0 0 1.57" />
-  </xacro:caster_wheel>
-  <xacro:caster_wheel name="mp_400_wheel_front_right" parent="base_footprint">
-    <origin xyz="0.164 -0.158 0.036" rpy="0 0 1.57" />
-  </xacro:caster_wheel>
-   <xacro:caster_wheel name="mp_400_wheel_back_right" parent="base_footprint">
-    <origin xyz="-0.319 -0.158 0.036" rpy="0 0 1.57" />
-  </xacro:caster_wheel>
-  <xacro:wheel_right name="mp_400_wheel_right" parent="base_footprint">
-    <origin xyz="0. -0.26 0.074" rpy="0 0 1.57" />
-  </xacro:wheel_right>
-  <xacro:wheel_left name="mp_400_wheel_left" parent="base_footprint">
-    <origin xyz="-0. 0.26 0.074" rpy="0 0 1.57" />
-  </xacro:wheel_left>
-  <!--+++++++++++++++++++laserscanner_link++++++++++++++++++++++++-->
-<!-- S300, NanoScan and Microscan -->
-  <xacro:sick_laser_v0 name="lidar_1" parent="base_link" ros_topic="lidar_1/scan_filtered">
-    <origin xyz="0.230 0 0.110" rpy="0 3.14 3.14" />
-  </xacro:sick_laser_v0>
-<!-- Igus -->
-<xacro:igus_5DOF_SV parent="base_link" prefix="igus">
-    <origin xyz="0 0 0." rpy="0 0 3.14" />
-  </xacro:igus_5DOF_SV>
-     <!--+++++++++++++++++++ IMU ++++++++++++++++++++++++-->
- <!-- Comment or uncomment based on your requirement -->
-<!--   <xacro:imu name="imu_1" parent="base_link">
-    <origin xyz="0.100 0 0.300" rpy="0 0 3.14" />
-  </xacro:imu> -->
-  <!--+++++++++++++++++++ Ultra Sonic ++++++++++++++++++++++++-->
-  <!-- Comment or uncomment based on your requirement -->
-  <!-- SENSOR 1 -->
-  <!-- xacro:us_sensor name="us_1" parent="base_link">
-    <origin xyz="0.100 0 0.300" rpy="0 3.14 3.14" />
-  </xacro:us_sensor-->
-  <!-- SENSOR 2 -->
-  <!-- xacro:us_sensor name="us_2" parent="base_link">
-    <origin xyz="0.110 0 0.300" rpy="0 3.14 3.14" />
-  </xacro:us_sensor-->
-  <!-- SENSOR 3 -->
-  <!-- xacro:us_sensor name="us_3" parent="base_link">
-    <origin xyz="0.120 0 0.300" rpy="0 3.14 3.14" />
-  </xacro:us_sensor-->
-  <!-- SENSOR 4 -->
-  <!-- xacro:us_sensor name="us_4" parent="base_link">
-    <origin xyz="0.130 0 0.300" rpy="0 3.14 3.14" />
-  </xacro:us_sensor-->
-  <!-- SENSOR 5 -->
-  <!-- xacro:us_sensor name="us_5" parent="base_link">
-    <origin xyz="0.140 0 0.300" rpy="0 3.14 3.14" />
-  </xacro:us_sensor-->
-  <!-- SENSOR 6 -->
-  <!-- xacro:us_sensor name="us_6" parent="base_link">
-    <origin xyz="0.150 0 0.300" rpy="0 3.14 3.14" />
-  </xacro:us_sensor-->
-  <!-- SENSOR 7 -->
-  <!-- xacro:us_sensor name="us_7" parent="base_link">
-    <origin xyz="0.160 0 0.300" rpy="0 3.14 3.14" />
-  </xacro:us_sensor-->
-  <!-- SENSOR 8 -->
-  <!-- xacro:us_sensor name="us_8" parent="base_link">
-    <origin xyz="0.170 0 0.300" rpy="0 3.14 3.14" />
-  </xacro:us_sensor-->
-  <!-- SENSOR 9 -->
-  <!-- xacro:us_sensor name="us_9" parent="base_link">
-    <origin xyz="0.180 0 0.300" rpy="0 3.14 3.14" />
-  </xacro:us_sensor-->
-  <!-- SENSOR 10 -->
-  <!-- xacro:us_sensor name="us_10" parent="base_link">
-    <origin xyz="0.100 0 0.300" rpy="0 3.14 3.14" />
-  </xacro:us_sensor-->
-  <!-- SENSOR 11 -->
-  <!-- xacro:us_sensor name="us_11" parent="base_link">
-    <origin xyz="0.100 0 0.300" rpy="0 3.14 3.14" />
-  </xacro:us_sensor-->
-  <!-- SENSOR 12 -->
-  <!-- xacro:us_sensor name="us_12" parent="base_link">
-    <origin xyz="0.190 0 0.300" rpy="0 3.14 3.14" />
-  </xacro:us_sensor-->
-  <!-- SENSOR 13 -->
-  <!-- xacro:us_sensor name="us_13" parent="base_link">
-    <origin xyz="0.200 0 0.300" rpy="0 3.14 3.14" />
-  </xacro:us_sensor-->
-  <!-- SENSOR 14 -->
-  <!-- xacro:us_sensor name="us_14" parent="base_link">
-    <origin xyz="0.210 0 0.300" rpy="0 3.14 3.14" />
-  </xacro:us_sensor-->
-  <!-- SENSOR 15 -->
-  <!-- xacro:us_sensor name="us_15" parent="base_link">
-    <origin xyz="0.220 0 0.300" rpy="0 3.14 3.14" />
-  </xacro:us_sensor-->
-  <!-- SENSOR 16 -->
-  <!-- xacro:us_sensor name="us_16" parent="base_link">
-    <origin xyz="0.230 0 0.300" rpy="0 3.14 3.14" />
-  </xacro:us_sensor-->
-    <!--Camera  -->
-<!-- <xacro:camera name="camera" parent="base_link">
-    <origin xyz="0 0 0.38" rpy="0 0 0" />
-  </xacro:camera> -->
+<robot xmlns:xacro="http://www.ros.org/wiki/xacro">
+  <xacro:macro name="igus_5DOF_SV" params="parent prefix *origin">
+    <joint name="linear_joint" type="fixed">
+      <parent link="${parent}" />
+      <child link = "linear_link" />
+      <origin xyz="0.0 0.0 0.375" rpy="-1.57 0.0 1.57" />
+      <axis xyz="0 0 1"/>
+      <limit effort="30" velocity="1.0" />
+    </joint>
+    <joint name="arm_joint" type="prismatic">
+      <parent link="linear_link" />
+      <child link = "igus_base_link" />
+      <origin xyz="0.0 -0.28 -0.0" rpy="3.14 0 1.57" />
+      <axis xyz="-1 0 0"/>
+      <limit effort="100" velocity="0.025" lower = "0.0" upper = "0.95"/>
+      <dynamics damping="1000.0"/>
+    </joint>
+    <link name="linear_link">
+    <visual>
+      <origin xyz="0.0 0.0 0.0" rpy="0 0 0"/>
+      <geometry>
+          <mesh filename="package://neo_mp_400/robot_model/mp_400/meshes/vertical_axis.dae"  scale="0.001 0.001 0.001"/>
+      </geometry>
+    </visual>
+    <collision>
+      <origin xyz="0.0 0.0 0.0" rpy="0 0 0"/>
+      <geometry>
+          <mesh filename="package://neo_mp_400/robot_model/mp_400/meshes/vertical_axis.dae"  scale="0.001 0.001 0.001"/>
+      </geometry>
+    </collision>
+     <inertial>
+      <origin xyz="0.0 0.0 0.0" rpy="0 0 0"/>
+      <mass value="30.0"/>
+      <inertia ixx="0.05" ixy="0.05" ixz="0.05" iyy="0.05" iyz="0.05" izz="0.05"/>
+    </inertial>
+  </link>
+  <link name="igus_base_link">
+    <visual>
+    <origin rpy="0 0 0" xyz="0 0 0"/>
+      <geometry>
+          <mesh filename="package://neo_mp_400/robot_model/mp_400/meshes/Joint0.dae"  scale="0.001 0.001 0.001"/>
+        </geometry>
+    </visual>
+    <collision>
+      <origin xyz="0 0 0" rpy="0 0 0" />
+      <geometry>
+          <mesh filename="package://neo_mp_400/robot_model/mp_400/meshes/Joint0.dae" scale="0.001 0.001 0.001"/>
+        </geometry>
+    </collision>
+    <inertial>
+      <origin xyz="0.0 0.0 0.0" rpy="0 0 0"/>
+      <mass value="5.0"/>
+      <inertia ixx="0.1045" ixy="-0.000460884801" ixz="0.000101130383"
+                    iyy="0.105" iyz="0.002941" izz="0.01284"/>
+    </inertial>
+  </link>
+  <link name="link1">
+    <visual>
+    <origin rpy="0 0 0" xyz="0.0 0 0.0"/>
+      <geometry>
+          <mesh filename="package://neo_mp_400/robot_model/mp_400/meshes/Joint1.dae"  scale="0.001 0.001 0.001"/>
+        </geometry>
+    </visual>
+    <collision>
+      <origin xyz="0 0 0" rpy="0 0 0" />
+      <geometry>
+          <mesh filename="package://neo_mp_400/robot_model/mp_400/meshes/Joint1.dae" scale="0.001 0.001 0.001"/>
+        </geometry>
+    </collision>
+<inertial>
+      <origin xyz="0.0 0.0 0.0" rpy="0 0 0"/>
+      <mass value="5.0"/>
+      <inertia ixx="0.1045" ixy="-0.000460884801" ixz="0.000101130383"
+                    iyy="0.105" iyz="0.002941" izz="0.01284"/>
+    </inertial>
+  </link>
+  <link name="link2">
+    <visual>
+    <origin rpy="0 0 0" xyz="0.0 0 0.0"/>
+      <geometry>
+          <mesh filename="package://neo_mp_400/robot_model/mp_400/meshes/Joint2.dae"  scale="0.001 0.001 0.001"/>
+        </geometry>
+    </visual>
+    <collision>
+      <origin xyz="0 0 0" rpy="0 0 0" />
+      <geometry>
+          <mesh filename="package://neo_mp_400/robot_model/mp_400/meshes/Joint2.dae" scale="0.001 0.001 0.001"/>
+        </geometry>
+    </collision>
+<inertial>
+      <origin xyz="0.0 0.0 0.0" rpy="0 0 0"/>
+      <mass value="5.0"/>
+      <inertia ixx="0.1045" ixy="-0.000460884801" ixz="0.000101130383"
+                    iyy="0.105" iyz="0.002941" izz="0.01284"/>
+    </inertial>
+  </link>
+  <link name="link3">
+    <visual>
+    <origin rpy="0 0 0" xyz="0.0 0 0"/>
+      <geometry>
+          <mesh filename="package://neo_mp_400/robot_model/mp_400/meshes/Joint3.dae"  scale="0.001 0.001 0.001"/>
+        </geometry>
+    </visual>
+    <collision>
+      <origin xyz="0 0 0" rpy="0 0 0" />
+      <geometry>
+          <mesh filename="package://neo_mp_400/robot_model/mp_400/meshes/Joint3.dae" scale="0.001 0.001 0.001"/>
+        </geometry>
+    </collision>
+  </link>
+  <link name="link4">
+    <visual>
+    <origin rpy="0 0 0" xyz="0.0 0 0.0"/>
+      <geometry>
+          <mesh filename="package://neo_mp_400/robot_model/mp_400/meshes/Joint4.dae"  scale="0.001 0.001 0.001"/>
+        </geometry>
+    </visual>
+    <collision>
+      <origin xyz="0 0 0" rpy="0 0 0" />
+      <geometry>
+          <mesh filename="package://neo_mp_400/robot_model/mp_400/meshes/Joint4.dae" scale="0.001 0.001 0.001"/>
+        </geometry>
+    </collision>
+  </link>
+  <link name="link5">
+    <visual>
+    <origin rpy="0 0 0" xyz="0 0 -0.0"/>
+      <geometry>
+          <mesh filename="package://neo_mp_400/robot_model/mp_400/meshes/Joint5.dae"  scale="0.001 0.001 0.001"/>
+        </geometry>
+    </visual>
+    <collision>
+      <origin xyz="0 0 0" rpy="0 0 -0.0" />
+      <geometry>
+          <mesh filename="package://neo_mp_400/robot_model/mp_400/meshes/Joint5.dae" scale="0.001 0.001 0.001"/>
+        </geometry>
+    </collision>
+  </link>
+  <link name="link6">
+    <visual>
+      <origin rpy="0.0 0 0" xyz="0 0 0"/>
+      <geometry>
+        <cylinder length="0.03" radius="0.035"/>
+      </geometry>
+    </visual>
+    <collision>
+      <origin xyz="0 0 0" rpy="0 0 -0.0" />
+      <geometry>
+        <cylinder length="0.03" radius="0.035"/>
+        </geometry>
+    </collision>
+  </link>
+  <joint name="joint1" type="revolute">
+    <axis xyz="0 0 1"/>
+    <parent link="igus_base_link"/>
+    <child link="link1"/>
+    <origin rpy="0 0 0" xyz="-0.05 0 0.185"/>
+      <limit effort="100" velocity="1.0" lower = "-2.53" upper = "2.53"/>
+    <joint_properties damping="0.0" friction="0.0"/>
+  </joint>
+ <joint name="joint2" type="revolute">
+    <axis xyz="0 1 0"/>
+    <parent link="link1"/>
+    <child link="link2"/>
+    <origin rpy="0 0 0" xyz="0 0 0.145"/>
+    <limit effort="100" lower="-0.785398" upper="1.22173" velocity="5"/>
+    <dynamics damping="15.0" friction="11"/>
+    <dynamics damping="100.0"/>
+  </joint>
+  <joint name="joint3" type="revolute">
+    <axis xyz="0 -1 0"/>
+    <parent link="link2"/>
+    <child link="link3"/>
+    <origin rpy="0 1.57079632679 0" xyz="0 0 0.350"/>
+    <limit effort="100" lower="-1.5708" upper="2.00713" velocity="5"/>
+    <dynamics damping="15.0" friction="11"/>
+  </joint>
+  <joint name="joint4" type="revolute">
+    <axis xyz="0 -1 0"/>
+    <parent link="link3"/>
+    <child link="link4"/>
+    <origin rpy="0 0 0" xyz="0 0 0.270"/>
+    <limit effort="100" lower="-0.523599" upper="2.0944" velocity="5"/>
+    <dynamics damping="15.0" friction="11"/>
+  </joint>
+  <joint name="joint5" type="revolute">
+    <axis xyz="0 0 1"/>
+    <parent link="link4"/>
+    <child link="link5"/>
+    <origin rpy="0 0 0" xyz="0 0 0.190"/>
+    <limit effort="100" lower="-0.174533" upper="0.174533" velocity="5"/>
+    <dynamics damping="15.0" friction="11"/>
+  </joint>
+ <joint name="joint6" type="revolute">
+    <axis xyz="0 0 1"/>
+    <parent link="link5"/>
+    <child link="link6"/>
+    <origin rpy="0 1.57 0" xyz="-0.04 0 0.04"/>
+      <limit effort="100" velocity="1.0" lower = "-3.14" upper = "3.14"/>
+    <joint_properties damping="0.0" friction="0.0"/>
+  </joint>
+    <transmission name="tran_prismatic">
+    <type>transmission_interface/SimpleTransmission</type>
+    <joint name="arm_joint">
+      <hardwareInterface>hardware_interface/VelocityJointInterface</hardwareInterface>
+    </joint>
+    <actuator name="tran_prismatic_motor">
+      <mechanicalReduction>15</mechanicalReduction>
+    </actuator>
+  </transmission>
+  <transmission name="tran_roll">
+    <type>transmission_interface/SimpleTransmission</type>
+    <joint name="joint1">
+      <hardwareInterface>hardware_interface/VelocityJointInterface</hardwareInterface>
+    </joint>
+    <actuator name="tran_roll_motor">
+      <mechanicalReduction>50</mechanicalReduction>
+    </actuator>
+  </transmission>
+  <transmission name="tran_1">
+    <type>transmission_interface/SimpleTransmission</type>
+    <joint name="joint2">
+      <hardwareInterface>hardware_interface/VelocityJointInterface</hardwareInterface>
+    </joint>
+    <actuator name="tran_1_motor">
+      <mechanicalReduction>50</mechanicalReduction>
+    </actuator>
+  </transmission>
+   <transmission name="tran_2">
+    <type>transmission_interface/SimpleTransmission</type>
+    <joint name="joint3">
+      <hardwareInterface>hardware_interface/VelocityJointInterface</hardwareInterface>
+    </joint>
+    <actuator name="tran_2_motor">
+      <mechanicalReduction>-38</mechanicalReduction>
+    </actuator>
+  </transmission>
+   <transmission name="tran_3">
+    <type>transmission_interface/SimpleTransmission</type>
+    <joint name="joint4">
+      <hardwareInterface>hardware_interface/VelocityJointInterface</hardwareInterface>
+    </joint>
+    <actuator name="tran_3_motor">
+      <mechanicalReduction>-38</mechanicalReduction>
+    </actuator>
+  </transmission>
+   <transmission name="tran_4">
+    <type>transmission_interface/SimpleTransmission</type>
+    <joint name="joint5">
+      <hardwareInterface>hardware_interface/VelocityJointInterface</hardwareInterface>
+    </joint>
+    <actuator name="tran_4_motor">
+      <mechanicalReduction>-28</mechanicalReduction>
+    </actuator>
+  </transmission>
+  <transmission name="tran_5">
+    <type>transmission_interface/SimpleTransmission</type>
+    <joint name="joint6">
+      <hardwareInterface>hardware_interface/VelocityJointInterface</hardwareInterface>
+    </joint>
+    <actuator name="tran_5_motor">
+      <mechanicalReduction>32</mechanicalReduction>
+    </actuator>
+  </transmission>
+    </xacro:macro>
 </robot>
